Commit message: prefer file:// over package://

File: spot_description/urdf/accessories.urdf.xacro (robot description, xacro)
@@ -10,15 +10,15 @@
       <visual>
         <geometry>
-          <mesh filename="package://spot_description/meshes/base/visual/pack_top.dae"/>
+          <mesh filename="file://$(find spot_description)/meshes/base/visual/pack_top.dae"/>
         </geometry>
       </visual>
       <visual>
         <geometry>
-          <mesh filename="package://spot_description/meshes/base/visual/pack_body.dae"/>
+          <mesh filename="file://$(find spot_description)/meshes/base/visual/pack_body.dae"/>
         </geometry>
       </visual>
       <collision>
         <geometry>
-          <mesh filename="package://spot_description/meshes/base/visual/pack_body.dae"/>
+          <mesh filename="file://$(find spot_description)/meshes/base/visual/pack_body.dae"/>
         </geometry>
       </collision>
@@ -34,10 +34,10 @@
       <visual>
         <geometry>
-          <mesh filename="package://spot_description/meshes/base/visual/lidar_mount.dae"/>
+          <mesh filename="file://$(find spot_description)/meshes/base/visual/lidar_mount.dae"/>
         </geometry>
       </visual>
       <collision>
         <geometry>
-          <mesh filename="package://spot_description/meshes/base/collision/lidar_mount_collision.stl"/>
+          <mesh filename="file://$(find spot_description)/meshes/base/collision/lidar_mount_collision.stl"/>
         </geometry>
       </collision>
@@ -53,5 +53,5 @@
         <visual>
           <geometry>
-            <mesh filename="package://spot_description/meshes/base/collision/velodyne_cage.stl" scale="0.001 0.001 0.001" />
+            <mesh filename="file://$(find spot_description)/meshes/base/collision/velodyne_cage.stl" scale="0.001 0.001 0.001" />
           </geometry>
           <origin xyz="0 0 0" rpy="0 0 0" />
@@ -60,5 +60,5 @@
         <collision>
           <geometry>
-            <mesh filename="package://spot_description/meshes/base/collision/velodyne_cage.stl" scale="0.001 0.001 0.001" />
+            <mesh filename="file://$(find spot_description)/meshes/base/collision/velodyne_cage.stl" scale="0.001 0.001 0.001" />
           </geometry>
           <origin xyz="0 0 0" rpy="0 0 0" />

File: spot_description/urdf/spot_macro.xacro (robot description, xacro)
@@ -7,10 +7,10 @@
             <visual>
                 <geometry>
-                    <mesh filename="package://spot_description/meshes/base/visual/body.dae" />
-                </geometry>
-            </visual>
-            <collision>
-                <geometry>
-                    <mesh filename="package://spot_description/meshes/base/collision/body_collision.stl" />
+                    <mesh filename="file://$(find spot_description)/meshes/base/visual/body.dae" />
+                </geometry>
+            </visual>
+            <collision>
+                <geometry>
+                    <mesh filename="file://$(find spot_description)/meshes/base/collision/body_collision.stl" />
                 </geometry>
             </collision>
@@ -55,10 +55,10 @@
             <visual>
                 <geometry>
-                    <mesh filename="package://spot_description/meshes/base/visual/front_left_hip.dae" />
-                </geometry>
-            </visual>
-            <collision>
-                <geometry>
-                    <mesh filename="package://spot_description/meshes/base/collision/front_left_hip_collision.stl" />
+                    <mesh filename="file://$(find spot_description)/meshes/base/visual/front_left_hip.dae" />
+                </geometry>
+            </visual>
+            <collision>
+                <geometry>
+                    <mesh filename="file://$(find spot_description)/meshes/base/collision/front_left_hip_collision.stl" />
                 </geometry>
             </collision>
@@ -79,10 +79,10 @@
             <visual>
                 <geometry>
-                    <mesh filename="package://spot_description/meshes/base/visual/front_left_upper_leg.dae" />
-                </geometry>
-            </visual>
-            <collision>
-                <geometry>
-                    <mesh filename="package://spot_description/meshes/base/collision/front_left_upper_leg_collision.stl" />
+                    <mesh filename="file://$(find spot_description)/meshes/base/visual/front_left_upper_leg.dae" />
+                </geometry>
+            </visual>
+            <collision>
+                <geometry>
+                    <mesh filename="file://$(find spot_description)/meshes/base/collision/front_left_upper_leg_collision.stl" />
                 </geometry>
             </collision>
@@ -103,10 +103,10 @@
             <visual>
                 <geometry>
-                    <mesh filename="package://spot_description/meshes/base/visual/front_left_lower_leg.dae" />
-                </geometry>
-            </visual>
-            <collision>
-                <geometry>
-                    <mesh filename="package://spot_description/meshes/base/collision/front_left_lower_leg_collision.stl" />
+                    <mesh filename="file://$(find spot_description)/meshes/base/visual/front_left_lower_leg.dae" />
+                </geometry>
+            </visual>
+            <collision>
+                <geometry>
+                    <mesh filename="file://$(find spot_description)/meshes/base/collision/front_left_lower_leg_collision.stl" />
                 </geometry>
             </collision>
@@ -127,10 +127,10 @@
             <visual>
                 <geometry>
-                    <mesh filename="package://spot_description/meshes/base/visual/front_right_hip.dae" />
-                </geometry>
-            </visual>
-            <collision>
-                <geometry>
-                    <mesh filename="package://spot_description/meshes/base/collision/front_right_hip_collision.stl" />
+                    <mesh filename="file://$(find spot_description)/meshes/base/visual/front_right_hip.dae" />
+                </geometry>
+            </visual>
+            <collision>
+                <geometry>
+                    <mesh filename="file://$(find spot_description)/meshes/base/collision/front_right_hip_collision.stl" />
                 </geometry>
             </collision>
@@ -151,10 +151,10 @@
             <visual>
                 <geometry>
-                    <mesh filename="package://spot_description/meshes/base/visual/front_right_upper_leg.dae" />
-                </geometry>
-            </visual>
-            <collision>
-                <geometry>
-                    <mesh filename="package://spot_description/meshes/base/collision/front_right_upper_leg_collision.stl" />
+                    <mesh filename="file://$(find spot_description)/meshes/base/visual/front_right_upper_leg.dae" />
+                </geometry>
+            </visual>
+            <collision>
+                <geometry>
+                    <mesh filename="file://$(find spot_description)/meshes/base/collision/front_right_upper_leg_collision.stl" />
                 </geometry>
             </collision>
@@ -175,10 +175,10 @@
             <visual>
                 <geometry>
-                    <mesh filename="package://spot_description/meshes/base/visual/front_right_lower_leg.dae" />
-                </geometry>
-            </visual>
-            <collision>
-                <geometry>
-                    <mesh filename="package://spot_description/meshes/base/collision/front_right_lower_leg_collision.stl" />
+                    <mesh filename="file://$(find spot_description)/meshes/base/visual/front_right_lower_leg.dae" />
+                </geometry>
+            </visual>
+            <collision>
+                <geometry>
+                    <mesh filename="file://$(find spot_description)/meshes/base/collision/front_right_lower_leg_collision.stl" />
                 </geometry>
             </collision>
@@ -199,10 +199,10 @@
             <visual>
                 <geometry>
-                    <mesh filename="package://spot_description/meshes/base/visual/rear_left_hip.dae" />
-                </geometry>
-            </visual>
-            <collision>
-                <geometry>
-                    <mesh filename="package://spot_description/meshes/base/collision/rear_left_hip_collision.stl" />
+                    <mesh filename="file://$(find spot_description)/meshes/base/visual/rear_left_hip.dae" />
+                </geometry>
+            </visual>
+            <collision>
+                <geometry>
+                    <mesh filename="file://$(find spot_description)/meshes/base/collision/rear_left_hip_collision.stl" />
                 </geometry>
             </collision>
@@ -223,10 +223,10 @@
             <visual>
                 <geometry>
-                    <mesh filename="package://spot_description/meshes/base/visual/rear_left_upper_leg.dae" />
-                </geometry>
-            </visual>
-            <collision>
-                <geometry>
-                    <mesh filename="package://spot_description/meshes/base/collision/rear_left_upper_leg_collision.stl" />
+                    <mesh filename="file://$(find spot_description)/meshes/base/visual/rear_left_upper_leg.dae" />
+                </geometry>
+            </visual>
+            <collision>
+                <geometry>
+                    <mesh filename="file://$(find spot_description)/meshes/base/collision/rear_left_upper_leg_collision.stl" />
                 </geometry>
             </collision>
@@ -247,10 +247,10 @@
             <visual>
                 <geometry>
-                    <mesh filename="package://spot_description/meshes/base/visual/rear_left_lower_leg.dae" />
-                </geometry>
-            </visual>
-            <collision>
-                <geometry>
-                    <mesh filename="package://spot_description/meshes/base/collision/rear_left_lower_leg_collision.stl" />
+                    <mesh filename="file://$(find spot_description)/meshes/base/visual/rear_left_lower_leg.dae" />
+                </geometry>
+            </visual>
+            <collision>
+                <geometry>
+                    <mesh filename="file://$(find spot_description)/meshes/base/collision/rear_left_lower_leg_collision.stl" />
                 </geometry>
             </collision>
@@ -271,10 +271,10 @@
             <visual>
                 <geometry>
-                    <mesh filename="package://spot_description/meshes/base/visual/rear_right_hip.dae" />
-                </geometry>
-            </visual>
-            <collision>
-                <geometry>
-                    <mesh filename="package://spot_description/meshes/base/collision/rear_right_hip_collision.stl" />
+                    <mesh filename="file://$(find spot_description)/meshes/base/visual/rear_right_hip.dae" />
+                </geometry>
+            </visual>
+            <collision>
+                <geometry>
+                    <mesh filename="file://$(find spot_description)/meshes/base/collision/rear_right_hip_collision.stl" />
                 </geometry>
             </collision>
@@ -295,10 +295,10 @@
             <visual>
                 <geometry>
-                    <mesh filename="package://spot_description/meshes/base/visual/rear_right_upper_leg.dae" />
-                </geometry>
-            </visual>
-            <collision>
-                <geometry>
-                    <mesh filename="package://spot_description/meshes/base/collision/rear_right_upper_leg_collision.stl" />
+                    <mesh filename="file://$(find spot_description)/meshes/base/visual/rear_right_upper_leg.dae" />
+                </geometry>
+            </visual>
+            <collision>
+                <geometry>
+                    <mesh filename="file://$(find spot_description)/meshes/base/collision/rear_right_upper_leg_collision.stl" />
                 </geometry>
             </collision>
@@ -319,10 +319,10 @@
             <visual>
                 <geometry>
-                    <mesh filename="package://spot_description/meshes/base/visual/rear_right_lower_leg.dae" />
-                </geometry>
-            </visual>
-            <collision>
-                <geometry>
-                    <mesh filename="package://spot_description/meshes/base/collision/rear_right_lower_leg_collision.stl" />
+                    <mesh filename="file://$(find spot_description)/meshes/base/visual/rear_right_lower_leg.dae" />
+                </geometry>
+            </visual>
+            <collision>
+                <geometry>
+                    <mesh filename="file://$(find spot_description)/meshes/base/collision/rear_right_lower_leg_collision.stl" />
                 </geometry>
             </collision>

File: spot_description/urdf/spot_simple.urdf.xacro (robot description, xacro)
@@ -5,5 +5,5 @@
       <origin xyz="0 0 0" rpy="0 0 0"/>
       <geometry>
-        <mesh filename="package://spot_description/meshes/base_simple/visual/body.obj"/>
+        <mesh filename="file://$(find spot_description)/meshes/base_simple/visual/body.obj"/>
       </geometry>
       <material name="body"> <color rgba="1 0.8431 0 1"/></material>
@@ -11,5 +11,5 @@
     <collision>
       <geometry>
-        <mesh filename="package://spot_description/meshes/base_simple/collision/body.stl" />
+        <mesh filename="file://$(find spot_description)/meshes/base_simple/collision/body.stl" />
       </geometry>
     </collision>
@@ -31,5 +31,5 @@
       <origin xyz="0 0 0" rpy="0 0 0"/>
       <geometry>
-        <mesh filename="package://spot_description/meshes/base_simple/visual/fl_hip.obj"/>
+        <mesh filename="file://$(find spot_description)/meshes/base_simple/visual/fl_hip.obj"/>
       </geometry>
       <material name="fl_hip"> <color rgba="0.2 0.2 0.2 1"/></material>
@@ -37,5 +37,5 @@
     <collision>
       <geometry>
-        <mesh filename="package://spot_description/meshes/base_simple/collision/fl_hip.stl" />
+        <mesh filename="file://$(find spot_description)/meshes/base_simple/collision/fl_hip.stl" />
       </geometry>
     </collision>
@@ -57,5 +57,5 @@
       <origin xyz="0 0 0" rpy="0 0 0"/>
       <geometry>
-        <mesh filename="package://spot_description/meshes/base_simple/visual/fl_uleg.obj"/>
+        <mesh filename="file://$(find spot_description)/meshes/base_simple/visual/fl_uleg.obj"/>
       </geometry>
       <material name="fl_uleg"> <color rgba="1 0.8431 0 1"/></material>
@@ -63,5 +63,5 @@
     <collision>
       <geometry>
-        <mesh filename="package://spot_description/meshes/base_simple/collision/fl_uleg.stl" />
+        <mesh filename="file://$(find spot_description)/meshes/base_simple/collision/fl_uleg.stl" />
       </geometry>
     </collision>
@@ -83,5 +83,5 @@
       <origin xyz="0 0 0" rpy="0 0 0"/>
       <geometry>
-        <mesh filename="package://spot_description/meshes/base_simple/visual/fl_lleg.obj"/>
+        <mesh filename="file://$(find spot_description)/meshes/base_simple/visual/fl_lleg.obj"/>
       </geometry>
       <material name="fl_lleg"> <color rgba="0.2 0.2 0.2 1"/></material>
@@ -89,5 +89,5 @@
     <collision>
       <geometry>
-        <mesh filename="package://spot_description/meshes/base_simple/collision/fl_lleg.stl" />
+        <mesh filename="file://$(find spot_description)/meshes/base_simple/collision/fl_lleg.stl" />
       </geometry>
     </collision>
@@ -109,5 +109,5 @@
       <origin xyz="0 0 0" rpy="0 0 0"/>
       <geometry>
-        <mesh filename="package://spot_description/meshes/base_simple/visual/fr_hip.obj"/>
+        <mesh filename="file://$(find spot_description)/meshes/base_simple/visual/fr_hip.obj"/>
       </geometry>
       <material name="fr_hip"> <color rgba="0.2 0.2 0.2 1"/></material>
@@ -115,5 +115,5 @@
     <collision>
       <geometry>
-        <mesh filename="package://spot_description/meshes/base_simple/collision/fr_hip.stl" />
+        <mesh filename="file://$(find spot_description)/meshes/base_simple/collision/fr_hip.stl" />
       </geometry>
     </collision>
@@ -135,5 +135,5 @@
       <origin xyz="0 0 0" rpy="0 0 0"/>
       <geometry>
-        <mesh filename="package://spot_description/meshes/base_simple/visual/fr_uleg.obj"/>
+        <mesh filename="file://$(find spot_description)/meshes/base_simple/visual/fr_uleg.obj"/>
       </geometry>
       <material name="fr_uleg"> <color rgba="1 0.8431 0 1"/></material>
@@ -141,5 +141,5 @@
     <collision>
       <geometry>
-        <mesh filename="package://spot_description/meshes/base_simple/collision/fr_uleg.stl" />
+        <mesh filename="file://$(find spot_description)/meshes/base_simple/collision/fr_uleg.stl" />
       </geometry>
     </collision>
@@ -161,5 +161,5 @@
       <origin xyz="0 0 0" rpy="0 0 0"/>
       <geometry>
-        <mesh filename="package://spot_description/meshes/base_simple/visual/fr_lleg.obj"/>
+        <mesh filename="file://$(find spot_description)/meshes/base_simple/visual/fr_lleg.obj"/>
       </geometry>
       <material name="fr_lleg"> <color rgba="0.2 0.2 0.2 1"/></material>
@@ -167,5 +167,5 @@
     <collision>
       <geometry>
-        <mesh filename="package://spot_description/meshes/base_simple/collision/fr_lleg.stl" />
+        <mesh filename="file://$(find spot_description)/meshes/base_simple/collision/fr_lleg.stl" />
       </geometry>
     </collision>
@@ -187,5 +187,5 @@
       <origin xyz="0 0 0" rpy="0 0 0"/>
       <geometry>
-        <mesh filename="package://spot_description/meshes/base_simple/visual/hl_hip.obj"/>
+        <mesh filename="file://$(find spot_description)/meshes/base_simple/visual/hl_hip.obj"/>
       </geometry>
       <material name="hl_hip"> <color rgba="0.2 0.2 0.2 1"/></material>
@@ -193,5 +193,5 @@
     <collision>
       <geometry>
-        <mesh filename="package://spot_description/meshes/base_simple/collision/hl_hip.stl" />
+        <mesh filename="file://$(find spot_description)/meshes/base_simple/collision/hl_hip.stl" />
       </geometry>
     </collision>
@@ -213,5 +213,5 @@
       <origin xyz="0 0 0" rpy="0 0 0"/>
       <geometry>
-        <mesh filename="package://spot_description/meshes/base_simple/visual/hl_uleg.obj"/>
+        <mesh filename="file://$(find spot_description)/meshes/base_simple/visual/hl_uleg.obj"/>
       </geometry>
       <material name="hl_uleg"> <color rgba="1 0.8431 0 1"/></material>
@@ -219,5 +219,5 @@
     <collision>
       <geometry>
-        <mesh filename="package://spot_description/meshes/base_simple/collision/hl_uleg.stl" />
+        <mesh filename="file://$(find spot_description)/meshes/base_simple/collision/hl_uleg.stl" />
       </geometry>
     </collision>
@@ -239,5 +239,5 @@
       <origin xyz="0 0 0" rpy="0 0 0"/>
       <geometry>
-        <mesh filename="package://spot_description/meshes/base_simple/visual/hl_lleg.obj"/>
+        <mesh filename="file://$(find spot_description)/meshes/base_simple/visual/hl_lleg.obj"/>
       </geometry>
       <material name="hl_lleg"> <color rgba="0.2 0.2 0.2 1"/></material>
@@ -245,5 +245,5 @@
     <collision>
       <geometry>
-        <mesh filename="package://spot_description/meshes/base_simple/collision/hl_lleg.stl" />
+        <mesh filename="file://$(find spot_description)/meshes/base_simple/collision/hl_lleg.stl" />
       </geometry>
     </collision>
@@ -265,5 +265,5 @@
       <origin xyz="0 0 0" rpy="0 0 0"/>
       <geometry>
-        <mesh filename="package://spot_description/meshes/base_simple/visual/hr_hip.obj"/>
+        <mesh filename="file://$(find spot_description)/meshes/base_simple/visual/hr_hip.obj"/>
       </geometry>
       <material name="hr_hip"> <color rgba="0.2 0.2 0.2 1"/></material>
@@ -271,5 +271,5 @@
     <collision>
       <geometry>
-        <mesh filename="package://spot_description/meshes/base_simple/collision/hr_hip.stl" />
+        <mesh filename="file://$(find spot_description)/meshes/base_simple/collision/hr_hip.stl" />
       </geometry>
     </collision>
@@ -291,5 +291,5 @@
       <origin xyz="0 0 0" rpy="0 0 0"/>
       <geometry>
-        <mesh filename="package://spot_description/meshes/base_simple/visual/hr_uleg.obj"/>
+        <mesh filename="file://$(find spot_description)/meshes/base_simple/visual/hr_uleg.obj"/>
       </geometry>
       <material name="hr_uleg"> <color rgba="1 0.8431 0 1"/></material>
@@ -297,5 +297,5 @@
     <collision>
       <geometry>
-        <mesh filename="package://spot_description/meshes/base_simple/collision/hr_uleg.stl" />
+        <mesh filename="file://$(find spot_description)/meshes/base_simple/collision/hr_uleg.stl" />
       </geometry>
     </collision>
@@ -317,5 +317,5 @@
       <origin xyz="0 0 0" rpy="0 0 0"/>
       <geometry>
-        <mesh filename="package://spot_description/meshes/base_simple/visual/hr_lleg.obj"/>
+        <mesh filename="file://$(find spot_description)/meshes/base_simple/visual/hr_lleg.obj"/>
       </geometry>
       <material name="hr_lleg"> <color rgba="0.2 0.2 0.2 1"/></material>
@@ -323,5 +323,5 @@
     <collision>
       <geometry>
-        <mesh filename="package://spot_description/meshes/base_simple/collision/hr_lleg.stl" />
+        <mesh filename="file://$(find spot_description)/meshes/base_simple/collision/hr_lleg.stl" />
       </geometry>
     </collision>
