Commit message: spot base inertias are corrected

File: spot_description/urdf/spot.urdf.xacro (robot description, xacro)
@@ -15,7 +15,7 @@
     <link name="base_link">
         <inertial>
-            <origin rpy="0.0 0.0 0.0" xyz="0.00192414 0.00131838 0.00063246"/>
-            <mass value="30.689437866210938"/>
-            <inertia ixx="0.18470187485218048" ixy="-0.0010424249339848757" ixz="0.016710679978132248" iyy="1.7260644435882568" iyz="-0.0006984919309616089" izz="1.7602781057357788"/>
+            <origin rpy="0.0 0.0 0.0" xyz="0.006394396536052227 -9.812158532440662e-05 0.0009113792330026627"/>
+            <mass value="32.86"/>
+            <inertia ixx="0.13143999874591827" ixy="0.0" ixz="0.0" iyy="0.13143999874591827" iyz="0.0" izz="0.13143999874591827"/>
         </inertial>
     </link>
@@ -61,7 +61,7 @@
         </collision>
         <inertial>
-            <origin rpy="0.0 0.0 0.0" xyz="-0.02228133  0.01223229 -0.00013698"/>
-            <mass value="1.4118226766586304"/>
-            <inertia ixx="0.002230902900919318" ixy="-0.00024908874183893204" ixz="-1.0821946489159018e-05" iyy="0.0032821425702422857" iyz="1.2908072676509619e-05" izz="0.0035330711398273706"/>
+            <origin rpy="-0.716521349312305 0.02956473059648479 0.03655230014702582" xyz="-0.005374345928430557 0.012841847725212574 9.875232353806496e-05"/>
+            <mass value="1.68"/>
+            <inertia ixx="0.0021147398873455382" ixy="0.0" ixz="0.0" iyy="0.0018129577956607131" iyz="0.0" izz="0.002265435737304666"/>
         </inertial>
     </link>
@@ -85,7 +85,7 @@
         </collision>
         <inertial>
-            <origin rpy="0.0 0.0 0.0" xyz="0.00579826 -0.00155725 -0.11736281"/>
-            <mass value="4.5664448738098145"/>
-            <inertia ixx="0.06118762493133545" ixy="-6.980347097851336e-05" ixz="0.0025271624326705933" iyy="0.05970980226993561" iyz="0.0020649367943406105" izz="0.008818766102194786"/>
+            <origin rpy="-0.26437828203369795 -0.04853174570753804 0.024046963096353124" xyz="0.005142373498529196 -0.0024323679972440004 -0.12100915610790253"/>
+            <mass value="2.34"/>
+            <inertia ixx="0.02755964961185679" ixy="0.0" ixz="0.0" iyy="0.027354914287651046" iyz="0.0" izz="0.002848145546743553"/>
         </inertial>
     </link>
@@ -109,7 +109,7 @@
         </collision>
         <inertial>
-            <origin rpy="0.0 0.0 0.0" xyz="0.00122378  0.00153545 -0.18036975"/>
-            <mass value="1.6851935386657715"/>
-            <inertia ixx="0.021835200488567352" ixy="-9.323281119577587e-06" ixz="0.0001474980526836589" iyy="0.0221591517329216" iyz="-3.458634819253348e-05" izz="0.0011837183265015483"/>
+            <origin rpy="-0.007266925694167092 -0.009591807116834161 0.00035255970529224356" xyz="0.00225794012658298 4.607596201822162e-05 -0.1800822913646698"/>
+            <mass value="0.35"/>
+            <inertia ixx="0.003999022654901177" ixy="0.0" ixz="0.0" iyy="0.0040503157598010785" iyz="0.0" izz="0.0001493402097647426"/>
         </inertial>
     </link>
@@ -133,7 +133,7 @@
         </collision>
         <inertial>
-            <origin rpy="0.0 0.0 0.0" xyz="-0.02265939 -0.01222293 -0.00025806"/>
-            <mass value="1.4104852676391602"/>
-            <inertia ixx="0.002241714159026742" ixy="0.0002604306791909039" ixz="-5.935402441537008e-06" iyy="0.0032587547320872545" iyz="-7.373964763246477e-06" izz="0.003521676640957594"/>
+            <origin rpy="0.7165213493123055 -0.02956473059648479 0.03655230014702582" xyz="-0.005374345928430557 -0.012841847725212574 -9.875232353806496e-05"/>
+            <mass value="1.68"/>
+            <inertia ixx="0.0021147398873455382" ixy="0.0" ixz="0.0" iyy="0.0018129577956607131" iyz="0.0" izz="0.002265435737304666"/>
         </inertial>
     </link>
@@ -157,7 +157,7 @@
         </collision>
         <inertial>
-            <origin rpy="0.0 0.0 0.0" xyz="0.00574215  0.00151489 -0.1176383"/>
-            <mass value="4.534761428833008"/>
-            <inertia ixx="0.06084978207945824" ixy="0.00016782207239884883" ixz="0.002611876232549548" iyy="0.05935850366950035" iyz="-0.0019535261671990156" izz="0.008716627024114132"/>
+            <origin rpy="0.2643905306958363 -0.04853174688302708 -0.024046943559834943" xyz="0.005142373498529196 0.0024323677644133568 -0.12100915610790253"/>
+            <mass value="2.34"/>
+            <inertia ixx="0.02755964678927691" ixy="0.0" ixz="0.0" iyy="0.02735491706466737" iyz="0.0" izz="0.0028481453594764797"/>
         </inertial>
     </link>
@@ -181,7 +181,7 @@
         </collision>
         <inertial>
-            <origin rpy="0.0 0.0 0.0" xyz="0.00159384 -0.00239605 -0.18014717"/>
-            <mass value="1.6578948497772217"/>
-            <inertia ixx="0.021659644320607185" ixy="-5.41498047823552e-06" ixz="0.00012902059825137258" iyy="0.02198193594813347" iyz="0.00011968409671681002" izz="0.0011500123655423522"/>
+            <origin rpy="-0.007266925694167092 -0.009591807116834161 0.00035255970529224356" xyz="0.00225794012658298 4.607596201822162e-05 -0.1800822913646698"/>
+            <mass value="0.35"/>
+            <inertia ixx="0.003999022654901177" ixy="0.0" ixz="0.0" iyy="0.0040503157598010785" iyz="0.0" izz="0.0001493402097647426"/>
         </inertial>
     </link>
@@ -205,7 +205,7 @@
         </collision>
         <inertial>
-            <origin rpy="0.0 0.0 0.0" xyz="0.02251509  0.01207632 -0.00010392"/>
-            <mass value="1.4201561212539673"/>
-            <inertia ixx="0.0022622011601924896" ixy="0.00024073614622466266" ixz="1.9728562620002776e-05" iyy="0.0033044079318642616" iyz="5.893074558116496e-06" izz="0.003563372418284416"/>
+            <origin rpy="0.7165213493123055 -0.02956473059648479 0.03655230014702582" xyz="-0.005374345928430557 -0.012841847725212574 -9.875232353806496e-05"/>
+            <mass value="1.68"/>
+            <inertia ixx="0.0021147398873455382" ixy="0.0" ixz="0.0" iyy="0.0018129577956607131" iyz="0.0" izz="0.002265435737304666"/>
         </inertial>
     </link>
@@ -229,7 +229,7 @@
         </collision>
         <inertial>
-            <origin rpy="0.0 0.0 0.0" xyz="0.00521431 -0.00158592 -0.11710322"/>
-            <mass value="4.536705493927002"/>
-            <inertia ixx="0.06095878407359123" ixy="-8.738194446777925e-05" ixz="0.002448485465720296" iyy="0.05945170670747757" iyz="0.0017479292582720518" izz="0.008690832182765007"/>
+            <origin rpy="-0.26437828203369795 -0.04853174570753804 0.024046963096353124" xyz="0.005142373498529196 -0.0024323679972440004 -0.12100915610790253"/>
+            <mass value="2.34"/>
+            <inertia ixx="0.02755964961185679" ixy="0.0" ixz="0.0" iyy="0.027354914287651046" iyz="0.0" izz="0.002848145546743553"/>
         </inertial>
     </link>
@@ -253,7 +253,7 @@
         </collision>
         <inertial>
-            <origin rpy="0.0 0.0 0.0" xyz="0.00093319  0.00145674 -0.17991927"/>
-            <mass value="1.6818592548370361"/>
-            <inertia ixx="0.02180398255586624" ixy="-5.7460838434053585e-06" ixz="0.00012676010373979807" iyy="0.022132718935608864" iyz="-1.6608482837909833e-05" izz="0.001179960323497653"/>
+            <origin rpy="-0.007266925694167092 -0.009591807116834161 0.00035255970529224356" xyz="0.00225794012658298 4.607596201822162e-05 -0.1800822913646698"/>
+            <mass value="0.35"/>
+            <inertia ixx="0.003999022654901177" ixy="0.0" ixz="0.0" iyy="0.0040503157598010785" iyz="0.0" izz="0.0001493402097647426"/>
         </inertial>
     </link>
@@ -277,7 +277,7 @@
         </collision>
         <inertial>
-            <origin rpy="0.0 0.0 0.0" xyz="2.2480870e-02 -1.2067979e-02 -9.2436501e-05"/>
-            <mass value="1.4211853742599487"/>
-            <inertia ixx="0.002264411421492696" ixy="-0.00023975687508936971" ixz="1.755120320012793e-05" iyy="0.003309530671685934" iyz="-5.547248292714357e-06" izz="0.0035681931767612696"/>
+            <origin rpy="0.7165213493123055 -0.02956473059648479 0.03655230014702582" xyz="-0.005374345928430557 -0.012841847725212574 -9.875232353806496e-05"/>
+            <mass value="1.68"/>
+            <inertia ixx="0.0021147398873455382" ixy="0.0" ixz="0.0" iyy="0.0018129577956607131" iyz="0.0" izz="0.002265435737304666"/>
         </inertial>
     </link>
@@ -301,7 +301,7 @@
         </collision>
         <inertial>
-            <origin rpy="0.0 0.0 0.0" xyz="0.00564834  0.00171534 -0.117723"/>
-            <mass value="4.532190322875977"/>
-            <inertia ixx="0.060795851051807404" ixy="0.00013766760821454227" ixz="0.0027449424378573895" iyy="0.05932316929101944" iyz="-0.0018466990441083908" izz="0.008713570423424244"/>
+            <origin rpy="0.2643905306958363 -0.04853174688302708 -0.024046943559834943" xyz="0.005142373498529196 0.0024323677644133568 -0.12100915610790253"/>
+            <mass value="2.34"/>
+            <inertia ixx="0.02755964678927691" ixy="0.0" ixz="0.0" iyy="0.02735491706466737" iyz="0.0" izz="0.0028481453594764797"/>
         </inertial>
     </link>
@@ -325,7 +325,7 @@
         </collision>
         <inertial>
-            <origin rpy="0.0 0.0 0.0" xyz="0.00123708 -0.00190588 -0.18145134"/>
-            <mass value="1.682421326637268"/>
-            <inertia ixx="0.02176680974662304" ixy="1.009165498544462e-05" ixz="0.00013806326023768634" iyy="0.022093402221798897" iyz="-4.056539182784036e-05" izz="0.0011830450966954231"/>
+            <origin rpy="-0.007266925694167092 -0.009591807116834161 0.00035255970529224356" xyz="0.00225794012658298 4.607596201822162e-05 -0.1800822913646698"/>
+            <mass value="0.35"/>
+            <inertia ixx="0.003999022654901177" ixy="0.0" ixz="0.0" iyy="0.0040503157598010785" iyz="0.0" izz="0.0001493402097647426"/>
         </inertial>
     </link>

File: spot_description/urdf/spot_simple.urdf.xacro (robot description, xacro)
@@ -17,7 +17,7 @@
   <link name="body_inertia">
     <inertial>
-      <origin rpy="-0.0008011562081029489 0.012186456056377803 -0.009867765251682314" xyz="0.006394396536052227 -9.812158532440662e-05 0.0009113792330026627"/>
-      <mass value="25.8173828125"/>
-      <inertia ixx="0.13859701543461675" ixy="0.0" ixz="0.0" iyy="1.3583116406027023" iyz="0.0" izz="1.3960145798559307"/>
+      <origin rpy="0.0 0.0 0.0" xyz="0.006394396536052227 -9.812158532440662e-05 0.0009113792330026627"/>
+      <mass value="32.86"/>
+      <inertia ixx="0.13143999874591827" ixy="0.0" ixz="0.0" iyy="0.13143999874591827" iyz="0.0" izz="0.13143999874591827"/>
     </inertial>
   </link>
@@ -42,6 +42,6 @@
     <inertial>
       <origin rpy="-0.716521349312305 0.02956473059648479 0.03655230014702582" xyz="-0.005374345928430557 0.012841847725212574 9.875232353806496e-05"/>
-      <mass value="0.6527733206748962"/>
-      <inertia ixx="0.0008216939096317348" ixy="0.0" ixz="0.0" iyy="0.0007044348079342571" iyz="0.0" izz="0.0008802475800196751"/>
+      <mass value="1.68"/>
+      <inertia ixx="0.0021147398873455382" ixy="0.0" ixz="0.0" iyy="0.0018129577956607131" iyz="0.0" izz="0.002265435737304666"/>
     </inertial>
   </link>
@@ -68,6 +68,6 @@
     <inertial>
       <origin rpy="-0.26437828203369795 -0.04853174570753804 0.024046963096353124" xyz="0.005142373498529196 -0.0024323679972440004 -0.12100915610790253"/>
-      <mass value="2.810458183288574"/>
-      <inertia ixx="0.033100530803357994" ixy="0.0" ixz="0.0" iyy="0.032854634023222015" iyz="0.0" izz="0.0034207664587417004"/>
+      <mass value="2.34"/>
+      <inertia ixx="0.02755964961185679" ixy="0.0" ixz="0.0" iyy="0.027354914287651046" iyz="0.0" izz="0.002848145546743553"/>
     </inertial>
   </link>
@@ -94,6 +94,6 @@
     <inertial>
       <origin rpy="-0.007266925694167092 -0.009591807116834161 0.00035255970529224356" xyz="0.00225794012658298 4.607596201822162e-05 -0.1800822913646698"/>
-      <mass value="0.9355916976928711"/>
-      <inertia ixx="0.01068986466242586" ixy="0.0" ixz="0.0" iyy="0.010826977131294028" iyz="0.0" izz="0.00039920415910127985"/>
+      <mass value="0.35"/>
+      <inertia ixx="0.003999022654901177" ixy="0.0" ixz="0.0" iyy="0.0040503157598010785" iyz="0.0" izz="0.0001493402097647426"/>
     </inertial>
   </link>
@@ -120,6 +120,6 @@
     <inertial>
       <origin rpy="0.7165213493123055 -0.02956473059648479 0.03655230014702582" xyz="-0.005374345928430557 -0.012841847725212574 -9.875232353806496e-05"/>
-      <mass value="0.6527733206748962"/>
-      <inertia ixx="0.0008216939096317348" ixy="0.0" ixz="0.0" iyy="0.0007044348079342571" iyz="0.0" izz="0.0008802475800196751"/>
+      <mass value="1.68"/>
+      <inertia ixx="0.0021147398873455382" ixy="0.0" ixz="0.0" iyy="0.0018129577956607131" iyz="0.0" izz="0.002265435737304666"/>
     </inertial>
   </link>
@@ -146,6 +146,6 @@
     <inertial>
       <origin rpy="0.2643905306958363 -0.04853174688302708 -0.024046943559834943" xyz="0.005142373498529196 0.0024323677644133568 -0.12100915610790253"/>
-      <mass value="2.810458183288574"/>
-      <inertia ixx="0.03310052806239654" ixy="0.0" ixz="0.0" iyy="0.0328546367134009" iyz="0.0" izz="0.0034207662766936446"/>
+      <mass value="2.34"/>
+      <inertia ixx="0.02755964678927691" ixy="0.0" ixz="0.0" iyy="0.02735491706466737" iyz="0.0" izz="0.0028481453594764797"/>
     </inertial>
   </link>
@@ -172,6 +172,6 @@
     <inertial>
       <origin rpy="-0.007266925694167092 -0.009591807116834161 0.00035255970529224356" xyz="0.00225794012658298 4.607596201822162e-05 -0.1800822913646698"/>
-      <mass value="0.9355916976928711"/>
-      <inertia ixx="0.01068986466242586" ixy="0.0" ixz="0.0" iyy="0.010826977131294028" iyz="0.0" izz="0.00039920415910127985"/>
+      <mass value="0.35"/>
+      <inertia ixx="0.003999022654901177" ixy="0.0" ixz="0.0" iyy="0.0040503157598010785" iyz="0.0" izz="0.0001493402097647426"/>
     </inertial>
   </link>
@@ -198,6 +198,6 @@
     <inertial>
       <origin rpy="0.7165213493123055 0.02956473059648479 -0.03655230014702582" xyz="0.005374345928430557 0.012841847725212574 -9.875232353806496e-05"/>
-      <mass value="0.6527733206748962"/>
-      <inertia ixx="0.0008216939096317348" ixy="0.0" ixz="0.0" iyy="0.0007044348079342571" iyz="0.0" izz="0.0008802475800196751"/>
+      <mass value="1.68"/>
+      <inertia ixx="0.0021147398873455382" ixy="0.0" ixz="0.0" iyy="0.0018129577956607131" iyz="0.0" izz="0.002265435737304666"/>
     </inertial>
   </link>
@@ -224,6 +224,6 @@
     <inertial>
       <origin rpy="-0.26437828203369795 -0.04853174570753804 0.024046963096353124" xyz="0.005142373498529196 -0.0024323679972440004 -0.12100915610790253"/>
-      <mass value="2.810458183288574"/>
-      <inertia ixx="0.033100530803357994" ixy="0.0" ixz="0.0" iyy="0.032854634023222015" iyz="0.0" izz="0.0034207664587417004"/>
+      <mass value="2.34"/>
+      <inertia ixx="0.02755964961185679" ixy="0.0" ixz="0.0" iyy="0.027354914287651046" iyz="0.0" izz="0.002848145546743553"/>
     </inertial>
   </link>
@@ -250,6 +250,6 @@
     <inertial>
       <origin rpy="-0.007266925694167092 -0.009591807116834161 0.00035255970529224356" xyz="0.00225794012658298 4.607596201822162e-05 -0.1800822913646698"/>
-      <mass value="0.9355916976928711"/>
-      <inertia ixx="0.01068986466242586" ixy="0.0" ixz="0.0" iyy="0.010826977131294028" iyz="0.0" izz="0.00039920415910127985"/>
+      <mass value="0.35"/>
+      <inertia ixx="0.003999022654901177" ixy="0.0" ixz="0.0" iyy="0.0040503157598010785" iyz="0.0" izz="0.0001493402097647426"/>
     </inertial>
   </link>
@@ -276,6 +276,6 @@
     <inertial>
       <origin rpy="-0.716521349312305 -0.02956473059648479 -0.03655230014702582" xyz="0.005374345928430557 -0.012841847725212574 9.875232353806496e-05"/>
-      <mass value="0.6527733206748962"/>
-      <inertia ixx="0.0008216939096317348" ixy="0.0" ixz="0.0" iyy="0.0007044348079342571" iyz="0.0" izz="0.0008802475800196751"/>
+      <mass value="1.68"/>
+      <inertia ixx="0.0021147398873455382" ixy="0.0" ixz="0.0" iyy="0.0018129577956607131" iyz="0.0" izz="0.002265435737304666"/>
     </inertial>
   </link>
@@ -302,6 +302,6 @@
     <inertial>
       <origin rpy="0.2643905306958363 -0.04853174688302708 -0.024046943559834943" xyz="0.005142373498529196 0.0024323677644133568 -0.12100915610790253"/>
-      <mass value="2.810458183288574"/>
-      <inertia ixx="0.03310052806239654" ixy="0.0" ixz="0.0" iyy="0.0328546367134009" iyz="0.0" izz="0.0034207662766936446"/>
+      <mass value="2.34"/>
+      <inertia ixx="0.02755964678927691" ixy="0.0" ixz="0.0" iyy="0.02735491706466737" iyz="0.0" izz="0.0028481453594764797"/>
     </inertial>
   </link>
@@ -328,6 +328,6 @@
     <inertial>
       <origin rpy="-0.007266925694167092 -0.009591807116834161 0.00035255970529224356" xyz="0.00225794012658298 4.607596201822162e-05 -0.1800822913646698"/>
-      <mass value="0.9355916976928711"/>
-      <inertia ixx="0.01068986466242586" ixy="0.0" ixz="0.0" iyy="0.010826977131294028" iyz="0.0" izz="0.00039920415910127985"/>
+      <mass value="0.35"/>
+      <inertia ixx="0.003999022654901177" ixy="0.0" ixz="0.0" iyy="0.0040503157598010785" iyz="0.0" izz="0.0001493402097647426"/>
     </inertial>
   </link>
