Commit message: Remove tf_prefix as it's no longer needed

File: spot_description/urdf/spot.urdf.xacro (robot description, xacro)
@@ -4,8 +4,6 @@
   <!-- Parameters -->
   <xacro:arg name="arm" default="false" />
-  <xacro:arg name="tf_prefix" default="" />
   <!-- Load Spot -->
   <xacro:load_spot
-    arm="$(arg arm)"
-    tf_prefix="$(arg tf_prefix)" />
+    arm="$(arg arm)" />
 </robot>

File: spot_description/urdf/spot_macro.xacro (robot description, xacro)
@@ -2,7 +2,6 @@
 <robot name="spot" xmlns:xacro="http://www.ros.org/wiki/xacro">
     <xacro:macro name="load_spot" params="
-    arm:=false
-    tf_prefix">
-        <link name="${tf_prefix}body">
+    arm:=false ">
+        <link name="body">
             <visual>
                 <geometry>
@@ -16,5 +15,5 @@
             </collision>
         </link>
-        <link name="${tf_prefix}base_link">
+        <link name="base_link">
             <inertial>
                 <origin rpy="0.0 0.0 0.0" xyz="0.006394396536052227 -9.812158532440662e-05 0.0009113792330026627"/>
@@ -23,10 +22,10 @@
             </inertial>
         </link>
-        <joint name="${tf_prefix}base_link_joint" type="fixed">
+        <joint name="base_link_joint" type="fixed">
             <origin xyz="0 0 0" rpy="0 0 0" />
-            <parent link="${tf_prefix}body" />
-            <child link="${tf_prefix}base_link" />
-        </joint>
-        <link name="${tf_prefix}front_rail">
+            <parent link="body" />
+            <child link="base_link" />
+        </joint>
+        <link name="front_rail">
             <inertial>
                 <origin rpy="0. 0. 0." xyz="0. 0. 0."/>
@@ -35,10 +34,10 @@
             </inertial>
         </link>
-        <joint name="${tf_prefix}front_rail_joint" type="fixed">
+        <joint name="front_rail_joint" type="fixed">
             <origin xyz="0.223 0 0.0805" rpy="0 0 0" />
-            <parent link="${tf_prefix}body" />
-            <child link="${tf_prefix}front_rail" />
-        </joint>
-        <link name="${tf_prefix}rear_rail">
+            <parent link="body" />
+            <child link="front_rail" />
+        </joint>
+        <link name="rear_rail">
             <inertial>
                 <origin rpy="0. 0. 0." xyz="0. 0. 0."/>
@@ -47,10 +46,10 @@
             </inertial>
         </link>
-        <joint name="${tf_prefix}rear_rail_joint" type="fixed">
+        <joint name="rear_rail_joint" type="fixed">
             <origin xyz="-0.223 0 0.0805" rpy="0 0 0" />
-            <parent link="${tf_prefix}body" />
-            <child link="${tf_prefix}rear_rail" />
-        </joint>
-        <link name="${tf_prefix}front_left_hip">
+            <parent link="body" />
+            <child link="rear_rail" />
+        </joint>
+        <link name="front_left_hip">
             <visual>
                 <geometry>
@@ -69,12 +68,12 @@
             </inertial>
         </link>
-        <joint name="${tf_prefix}front_left_hip_x" type="revolute">
+        <joint name="front_left_hip_x" type="revolute">
             <origin xyz="0.29785 0.05500 0.00000" rpy="0 0 0" />
             <axis xyz="1 0 0" />
-            <parent link="${tf_prefix}body" />
-            <child link="${tf_prefix}front_left_hip" />
+            <parent link="body" />
+            <child link="front_left_hip" />
             <limit effort="1000" velocity="1000.00" lower="-0.78539816339744827899" upper="0.78539816339744827899" />
         </joint>
-        <link name="${tf_prefix}front_left_upper_leg">
+        <link name="front_left_upper_leg">
             <visual>
                 <geometry>
@@ -93,12 +92,12 @@
             </inertial>
         </link>
-        <joint name="${tf_prefix}front_left_hip_y" type="revolute">
+        <joint name="front_left_hip_y" type="revolute">
             <origin xyz="0.0 0.110945 0.0" rpy="0 0 0" />
             <axis xyz="0 1 0" />
-            <parent link="${tf_prefix}front_left_hip" />
-            <child link="${tf_prefix}front_left_upper_leg" />
+            <parent link="front_left_hip" />
+            <child link="front_left_upper_leg" />
             <limit effort="1000" velocity="1000.00" lower="-0.89884456477707963539" upper="2.2951079663725435509" />
         </joint>
-        <link name="${tf_prefix}front_left_lower_leg">
+        <link name="front_left_lower_leg">
             <visual>
                 <geometry>
@@ -117,12 +116,12 @@
             </inertial>
         </link>
-        <joint name="${tf_prefix}front_left_knee" type="revolute">
+        <joint name="front_left_knee" type="revolute">
             <origin xyz="0.025 0.000 -0.3205" rpy="0 0 0" />
             <axis xyz="0 1 0" />
-            <parent link="${tf_prefix}front_left_upper_leg" />
-            <child link="${tf_prefix}front_left_lower_leg" />
+            <parent link="front_left_upper_leg" />
+            <child link="front_left_lower_leg" />
             <limit effort="1000" velocity="1000.00" lower="-2.7929" upper="-0.254801" />
         </joint>
-        <link name="${tf_prefix}front_right_hip">
+        <link name="front_right_hip">
             <visual>
                 <geometry>
@@ -141,12 +140,12 @@
             </inertial>
         </link>
-        <joint name="${tf_prefix}front_right_hip_x" type="revolute">
+        <joint name="front_right_hip_x" type="revolute">
             <origin xyz="0.29785 -0.05500 0.00000" rpy="0 0 0" />
             <axis xyz="1 0 0" />
-            <parent link="${tf_prefix}body" />
-            <child link="${tf_prefix}front_right_hip" />
+            <parent link="body" />
+            <child link="front_right_hip" />
             <limit effort="1000" velocity="1000.00" lower="-0.78539816339744827899" upper="0.78539816339744827899" />
         </joint>
-        <link name="${tf_prefix}front_right_upper_leg">
+        <link name="front_right_upper_leg">
             <visual>
                 <geometry>
@@ -165,12 +164,12 @@
             </inertial>
         </link>
-        <joint name="${tf_prefix}front_right_hip_y" type="revolute">
+        <joint name="front_right_hip_y" type="revolute">
             <origin xyz="0.0 -0.110945 0.0" rpy="0 0 0" />
             <axis xyz="0 1 0" />
-            <parent link="${tf_prefix}front_right_hip" />
-            <child link="${tf_prefix}front_right_upper_leg" />
+            <parent link="front_right_hip" />
+            <child link="front_right_upper_leg" />
             <limit effort="1000" velocity="1000.00" lower="-0.89884456477707963539" upper="2.2951079663725435509" />
         </joint>
-        <link name="${tf_prefix}front_right_lower_leg">
+        <link name="front_right_lower_leg">
             <visual>
                 <geometry>
@@ -189,12 +188,12 @@
             </inertial>
         </link>
-        <joint name="${tf_prefix}front_right_knee" type="revolute">
+        <joint name="front_right_knee" type="revolute">
             <origin xyz="0.025 0.000 -0.3205" rpy="0 0 0" />
             <axis xyz="0 1 0" />
-            <parent link="${tf_prefix}front_right_upper_leg" />
-            <child link="${tf_prefix}front_right_lower_leg" />
+            <parent link="front_right_upper_leg" />
+            <child link="front_right_lower_leg" />
             <limit effort="1000" velocity="1000.00" lower="-2.7929" upper="-0.247563" />
         </joint>
-        <link name="${tf_prefix}rear_left_hip">
+        <link name="rear_left_hip">
             <visual>
                 <geometry>
@@ -213,12 +212,12 @@
             </inertial>
         </link>
-        <joint name="${tf_prefix}rear_left_hip_x" type="revolute">
+        <joint name="rear_left_hip_x" type="revolute">
             <origin xyz="-0.29785 0.05500 0.00000" rpy="0 0 0" />
             <axis xyz="1 0 0" />
-            <parent link="${tf_prefix}body" />
-            <child link="${tf_prefix}rear_left_hip" />
+            <parent link="body" />
+            <child link="rear_left_hip" />
             <limit effort="1000" velocity="1000.00" lower="-0.78539816339744827899" upper="0.78539816339744827899" />
         </joint>
-        <link name="${tf_prefix}rear_left_upper_leg">
+        <link name="rear_left_upper_leg">
             <visual>
                 <geometry>
@@ -237,12 +236,12 @@
             </inertial>
         </link>
-        <joint name="${tf_prefix}rear_left_hip_y" type="revolute">
+        <joint name="rear_left_hip_y" type="revolute">
             <origin xyz="0.0 0.110945 0.0" rpy="0 0 0" />
             <axis xyz="0 1 0" />
-            <parent link="${tf_prefix}rear_left_hip" />
-            <child link="${tf_prefix}rear_left_upper_leg" />
+            <parent link="rear_left_hip" />
+            <child link="rear_left_upper_leg" />
             <limit effort="1000" velocity="1000.00" lower="-0.89884456477707963539" upper="2.2951079663725435509" />
         </joint>
-        <link name="${tf_prefix}rear_left_lower_leg">
+        <link name="rear_left_lower_leg">
             <visual>
                 <geometry>
@@ -261,12 +260,12 @@
             </inertial>
         </link>
-        <joint name="${tf_prefix}rear_left_knee" type="revolute">
+        <joint name="rear_left_knee" type="revolute">
             <origin xyz="0.025 0.000 -0.3205" rpy="0 0 0" />
             <axis xyz="0 1 0" />
-            <parent link="${tf_prefix}rear_left_upper_leg" />
-            <child link="${tf_prefix}rear_left_lower_leg" />
+            <parent link="rear_left_upper_leg" />
+            <child link="rear_left_lower_leg" />
             <limit effort="1000" velocity="1000.00" lower="-2.7929" upper="-0.267153" />
         </joint>
-        <link name="${tf_prefix}rear_right_hip">
+        <link name="rear_right_hip">
             <visual>
                 <geometry>
@@ -285,12 +284,12 @@
             </inertial>
         </link>
-        <joint name="${tf_prefix}rear_right_hip_x" type="revolute">
+        <joint name="rear_right_hip_x" type="revolute">
             <origin xyz="-0.29785 -0.05500 0.00000" rpy="0 0 0" />
             <axis xyz="1 0 0" />
-            <parent link="${tf_prefix}body" />
-            <child link="${tf_prefix}rear_right_hip" />
+            <parent link="body" />
+            <child link="rear_right_hip" />
             <limit effort="1000" velocity="1000.00" lower="-0.78539816339744827899" upper="0.78539816339744827899" />
         </joint>
-        <link name="${tf_prefix}rear_right_upper_leg">
+        <link name="rear_right_upper_leg">
             <visual>
                 <geometry>
@@ -309,12 +308,12 @@
             </inertial>
         </link>
-        <joint name="${tf_prefix}rear_right_hip_y" type="revolute">
+        <joint name="rear_right_hip_y" type="revolute">
             <origin xyz="0.0 -0.110945 0.0" rpy="0 0 0" />
             <axis xyz="0 1 0" />
-            <parent link="${tf_prefix}rear_right_hip" />
-            <child link="${tf_prefix}rear_right_upper_leg" />
+            <parent link="rear_right_hip" />
+            <child link="rear_right_upper_leg" />
             <limit effort="1000" velocity="1000.00" lower="-0.89884456477707963539" upper="2.2951079663725435509" />
         </joint>
-        <link name="${tf_prefix}rear_right_lower_leg">
+        <link name="rear_right_lower_leg">
             <visual>
                 <geometry>
@@ -333,9 +332,9 @@
             </inertial>
         </link>
-        <joint name="${tf_prefix}rear_right_knee" type="revolute">
+        <joint name="rear_right_knee" type="revolute">
             <origin xyz="0.025 0.000 -0.3205" rpy="0 0 0" />
             <axis xyz="0 1 0" />
-            <parent link="${tf_prefix}rear_right_upper_leg" />
-            <child link="${tf_prefix}rear_right_lower_leg" />
+            <parent link="rear_right_upper_leg" />
+            <child link="rear_right_lower_leg" />
             <limit effort="1000" velocity="1000.00" lower="-2.7929" upper="-0.257725" />
         </joint>
@@ -347,5 +346,5 @@
         <xacro:if value="${arm}">
             <xacro:include filename="$(find spot_description)/urdf/spot_arm_macro.urdf" />
-            <xacro:load_arm tf_prefix="${tf_prefix}" />
+            <xacro:load_arm />
         </xacro:if>
     </xacro:macro>
