Commit message: Can correctly generate a urdf with tags

File: spot_description/urdf/spot_macro.xacro (robot description, xacro)
@@ -402,5 +402,6 @@
         <xacro:include filename="$(find spot_description)/urdf/accessories.urdf.xacro" />
         <!-- Optional custom includes. -->
-        <xacro:include filename="$(optenv SPOT_URDF_EXTRAS empty.urdf)" />
+        <xacro:property name="default_empty_urdf" value="$(find spot_description)/urdf/empty.urdf" />
+        <xacro:include filename="$(optenv SPOT_URDF_EXTRAS ${default_empty_urdf})" />
         <!-- Include Arm if necessary-->
         <xacro:if value="${arm}">

File: spot_ros2_control/xacro/spot_body.xacro (robot description, xacro)
@@ -12,10 +12,10 @@
     <xacro:include filename="$(find spot_description)/urdf/spot.urdf.xacro" />
     <xacro:include filename="$(find spot_ros2_control)/xacro/spot_interfaces.ros2_control.xacro" />
-    <xacro:include filename="$(find h1_description)/xacro/spot.ros2_control.xacro" />
+    <xacro:include filename="$(find spot_ros2_control)/xacro/spot.ros2_control.xacro" />
     <!-- Adding Spot-->
-    <xacro:spot />
+    <xacro:load_spot arm="false" tf_prefix=""/>
     <!-- Adding the ros2control tags without hands-->
     <xacro:if value="${add_ros2control_tag_property}">
-        <xacro:spot_ros2_control />
+        <!-- <xacro:spot_ros2_control /> -->
         <xacro:spot_interface_ros2_control />
     </xacro:if>

File: spot_ros2_control/xacro/spot_interfaces.ros2_control.xacro (robot description, xacro)
@@ -44,9 +44,9 @@
     </xacro:macro>
     <xacro:macro name="leg" params="left_or_right front_or_back">
-        <xacro:ros2control_joint joint_name="${front_or_back}_{left_or_right}_hip_x"
+        <xacro:ros2control_joint joint_name="${front_or_back}_${left_or_right}_hip_x"
             position_min="-0.785" position_max="0.785" velocity_max="100" effort_max="100" />
-        <xacro:ros2control_joint joint_name="${front_or_back}_{left_or_right}_hip_y"
+        <xacro:ros2control_joint joint_name="${front_or_back}_${left_or_right}_hip_y"
             position_min="-0.899" position_max="2.295" velocity_max="100" effort_max="100" />
-        <xacro:ros2control_joint joint_name="${front_or_back}_{left_or_right}_knee"
+        <xacro:ros2control_joint joint_name="${front_or_back}_${left_or_right}_knee"
             position_min="-2.793" position_max="-0.255" velocity_max="100" effort_max="100" />
     </xacro:macro>

Commit message: Update velocity values with more reasonable values from BD

File: spot_description/urdf/spot_macro.xacro (robot description, xacro)
@@ -76,5 +76,5 @@
             <parent link="${tf_prefix}body" />
             <child link="${tf_prefix}front_left_hip" />
-            <limit effort="45" velocity="1000.00" lower="-0.78539816339744827899"
+            <limit effort="45" velocity="17.647" lower="-0.78539816339744827899"
                 upper="0.78539816339744827899" />
         </joint>
@@ -105,5 +105,5 @@
             <parent link="${tf_prefix}front_left_hip" />
             <child link="${tf_prefix}front_left_upper_leg" />
-            <limit effort="45" velocity="1000.00" lower="-0.89884456477707963539"
+            <limit effort="45" velocity="17.647" lower="-0.89884456477707963539"
                 upper="2.2951079663725435509" />
         </joint>
@@ -140,5 +140,5 @@
             <parent link="${tf_prefix}front_left_upper_leg" />
             <child link="${tf_prefix}front_left_lower_leg" />
-            <limit effort="115" velocity="1000.00" lower="-2.7929" upper="-0.254801" />
+            <limit effort="115" velocity="12.0" lower="-2.7929" upper="-0.254801" />
         </joint>
         <link name="${tf_prefix}front_right_hip">
@@ -162,5 +162,5 @@
             <parent link="${tf_prefix}body" />
             <child link="${tf_prefix}front_right_hip" />
-            <limit effort="45" velocity="1000.00" lower="-0.78539816339744827899"
+            <limit effort="45" velocity="17.647" lower="-0.78539816339744827899"
                 upper="0.78539816339744827899" />
         </joint>
@@ -191,5 +191,5 @@
             <parent link="${tf_prefix}front_right_hip" />
             <child link="${tf_prefix}front_right_upper_leg" />
-            <limit effort="45" velocity="1000.00" lower="-0.89884456477707963539"
+            <limit effort="45" velocity="17.647" lower="-0.89884456477707963539"
                 upper="2.2951079663725435509" />
         </joint>
@@ -226,5 +226,5 @@
             <parent link="${tf_prefix}front_right_upper_leg" />
             <child link="${tf_prefix}front_right_lower_leg" />
-            <limit effort="115" velocity="1000.00" lower="-2.7929" upper="-0.247563" />
+            <limit effort="115" velocity="12.0" lower="-2.7929" upper="-0.247563" />
         </joint>
         <link name="${tf_prefix}rear_left_hip">
@@ -248,5 +248,5 @@
             <parent link="${tf_prefix}body" />
             <child link="${tf_prefix}rear_left_hip" />
-            <limit effort="45" velocity="1000.00" lower="-0.78539816339744827899"
+            <limit effort="45" velocity="17.647" lower="-0.78539816339744827899"
                 upper="0.78539816339744827899" />
         </joint>
@@ -277,5 +277,5 @@
             <parent link="${tf_prefix}rear_left_hip" />
             <child link="${tf_prefix}rear_left_upper_leg" />
-            <limit effort="45" velocity="1000.00" lower="-0.89884456477707963539"
+            <limit effort="45" velocity="17.647" lower="-0.89884456477707963539"
                 upper="2.2951079663725435509" />
         </joint>
@@ -312,5 +312,5 @@
             <parent link="${tf_prefix}rear_left_upper_leg" />
             <child link="${tf_prefix}rear_left_lower_leg" />
-            <limit effort="115" velocity="1000.00" lower="-2.7929" upper="-0.267153" />
+            <limit effort="115" velocity="12.0" lower="-2.7929" upper="-0.267153" />
         </joint>
         <link name="${tf_prefix}rear_right_hip">
@@ -334,5 +334,5 @@
             <parent link="${tf_prefix}body" />
             <child link="${tf_prefix}rear_right_hip" />
-            <limit effort="45" velocity="1000.00" lower="-0.78539816339744827899"
+            <limit effort="45" velocity="17.647" lower="-0.78539816339744827899"
                 upper="0.78539816339744827899" />
         </joint>
@@ -363,5 +363,5 @@
             <parent link="${tf_prefix}rear_right_hip" />
             <child link="${tf_prefix}rear_right_upper_leg" />
-            <limit effort="45" velocity="1000.00" lower="-0.89884456477707963539"
+            <limit effort="45" velocity="17.647" lower="-0.89884456477707963539"
                 upper="2.2951079663725435509" />
         </joint>
@@ -398,5 +398,5 @@
             <parent link="${tf_prefix}rear_right_upper_leg" />
             <child link="${tf_prefix}rear_right_lower_leg" />
-            <limit effort="115" velocity="1000.00" lower="-2.7929" upper="-0.257725" />
+            <limit effort="115" velocity="12.0" lower="-2.7929" upper="-0.257725" />
         </joint>
         <!-- Standard accessories. -->

Commit message: Dev/ros2 control (#471)
Co-authored-by: Katie Hughes <157421702+khughes-bdai@users.noreply.github.com>
Co-authored-by: Katie Hughes <khughes-bdai@theaiinstitute.com>
Co-authored-by: Laura Lee <129791566+llee-bdai@users.noreply.github.com>
Co-authored-by: Andrew Messing <129519955+amessing-bdai@users.noreply.github.com>

File: spot_description/urdf/spot_macro.xacro (robot description, xacro)
@@ -403,5 +403,6 @@
         <xacro:include filename="$(find spot_description)/urdf/accessories.urdf.xacro" />
         <!-- Optional custom includes. -->
-        <xacro:include filename="$(optenv SPOT_URDF_EXTRAS empty.urdf)" />
+        <xacro:property name="default_empty_urdf" value="$(find spot_description)/urdf/empty.urdf" />
+        <xacro:include filename="$(optenv SPOT_URDF_EXTRAS ${default_empty_urdf})" />
         <!-- Include Arm if necessary-->
         <xacro:if value="${arm}">
