Commit message: Move xacros to spot description

File: spot_description/urdf/spot.ros2_control.xacro (robot description, xacro)
@@ -52,3 +52,31 @@
             position_min="-1.570" position_max="0.000" velocity_max="100" effort_max="15.3" />
     </xacro:macro>
+    <xacro:macro name="spot_ros2_control" params="interface_type has_arm hostname username password tf_prefix">
+        <!-- Currently implements a simple system interface that covers all joints of the robot.
+        In the future, we could make different hardware interfaces for the body, arm, etc. -->
+        <ros2_control name="SpotSystem" type="system">
+            <hardware>
+            <xacro:if value="${interface_type == 'mock'}">
+                <plugin>mock_components/GenericSystem</plugin>
+                <param name="mock_sensor_commands">false</param>
+                <param name="state_following_offset">0.0</param>
+            </xacro:if>
+            <xacro:if value="${interface_type == 'robot'}">
+                <plugin>spot_ros2_control/SpotHardware</plugin>
+                <param name="hostname">$(optenv SPOT_IP ${hostname})</param>
+                <param name="username">$(optenv BOSDYN_CLIENT_USERNAME ${username})</param>
+                <param name="password">$(optenv BOSDYN_CLIENT_PASSWORD ${password})</param>
+            </xacro:if>
+            </hardware>
+            <!-- Add the legs -->
+            <xacro:leg front_or_rear="front" left_or_right="left" tf_prefix="${tf_prefix}" />
+            <xacro:leg front_or_rear="front" left_or_right="right" tf_prefix="${tf_prefix}" />
+            <xacro:leg front_or_rear="rear" left_or_right="left" tf_prefix="${tf_prefix}" />
+            <xacro:leg front_or_rear="rear" left_or_right="right" tf_prefix="${tf_prefix}" />
+            <!-- Add the arm + the gripper if the robot has an arm -->
+            <xacro:if value="${has_arm}">
+                <xacro:arm tf_prefix="${tf_prefix}" />
+            </xacro:if>
+        </ros2_control>
+    </xacro:macro>
 </robot>

Commit message: Baseline passing array into hardware interface

File: spot_description/urdf/spot.ros2_control.xacro (robot description, xacro)
@@ -19,8 +19,4 @@
                 <param name="max">${effort_max}</param>
             </command_interface>
-            <!-- TODO at some point, this should be a part of the command interface so we can have a
-            one-to-one mapping to the spot sdk implementation. -->
-            <!-- <command_interface name="k_q_p" />
-            <command_interface name="k_qd_p" /> -->
         </joint>
     </xacro:macro>
@@ -52,5 +48,5 @@
             position_min="-1.570" position_max="0.000" velocity_max="100" effort_max="15.3" />
     </xacro:macro>
-    <xacro:macro name="spot_ros2_control" params="interface_type has_arm hostname username password tf_prefix">
+    <xacro:macro name="spot_ros2_control" params="interface_type has_arm hostname username password tf_prefix kp kd">
         <!-- Currently implements a simple system interface that covers all joints of the robot.
         In the future, we could make different hardware interfaces for the body, arm, etc. -->
@@ -67,4 +63,6 @@
                 <param name="username">$(optenv BOSDYN_CLIENT_USERNAME ${username})</param>
                 <param name="password">$(optenv BOSDYN_CLIENT_PASSWORD ${password})</param>
+                <param name="kp">${kp}</param>
+                <param name="kd">${kd}</param>
             </xacro:if>
             </hardware>

File: spot_description/urdf/spot.urdf.xacro (robot description, xacro)
@@ -12,8 +12,9 @@
   <xacro:arg name="add_ros2_control_tag" default="false" />
   <xacro:arg name="hardware_interface_type" default="mock" />
-  <xacro:arg name="tf_prefix" default="" />
   <xacro:arg name="hostname" default="10.0.0.3" />
   <xacro:arg name="username" default="username" />
   <xacro:arg name="password" default="password" />
+  <xacro:arg name="kp" default="" />
+  <xacro:arg name="kd" default="" />
   <!-- Load Spot -->
   <xacro:load_spot
@@ -28,5 +29,7 @@
                                username="$(arg username)"
                                password="$(arg password)"
-                               tf_prefix="$(arg tf_prefix)" />
+                               tf_prefix="$(arg tf_prefix)"
+                               kd="$(arg kd)"
+                               kp="$(arg kp)" />
   </xacro:if>
 </robot>

Commit message: Mass change variable names to match bd convention

File: spot_description/urdf/spot.ros2_control.xacro (robot description, xacro)
@@ -48,5 +48,5 @@
             position_min="-1.570" position_max="0.000" velocity_max="100" effort_max="15.3" />
     </xacro:macro>
-    <xacro:macro name="spot_ros2_control" params="interface_type has_arm hostname username password tf_prefix kp kd">
+    <xacro:macro name="spot_ros2_control" params="interface_type has_arm hostname username password tf_prefix k_q_p k_qd_p">
         <!-- Currently implements a simple system interface that covers all joints of the robot.
         In the future, we could make different hardware interfaces for the body, arm, etc. -->
@@ -63,6 +63,6 @@
                 <param name="username">$(optenv BOSDYN_CLIENT_USERNAME ${username})</param>
                 <param name="password">$(optenv BOSDYN_CLIENT_PASSWORD ${password})</param>
-                <param name="kp">${kp}</param>
-                <param name="kd">${kd}</param>
+                <param name="k_q_p">${k_q_p}</param>
+                <param name="k_qd_p">${k_qd_p}</param>
             </xacro:if>
             </hardware>

File: spot_description/urdf/spot.urdf.xacro (robot description, xacro)
@@ -15,6 +15,6 @@
   <xacro:arg name="username" default="username" />
   <xacro:arg name="password" default="password" />
-  <xacro:arg name="kp" default="" />
-  <xacro:arg name="kd" default="" />
+  <xacro:arg name="k_q_p" default="" />
+  <xacro:arg name="k_qd_p" default="" />
   <!-- Load Spot -->
   <xacro:load_spot
@@ -30,6 +30,6 @@
                                password="$(arg password)"
                                tf_prefix="$(arg tf_prefix)"
-                               kd="$(arg kd)"
-                               kp="$(arg kp)" />
+                               k_q_p="$(arg k_q_p)"
+                               k_qd_p="$(arg k_qd_p)" />
   </xacro:if>
 </robot>

Commit message: [SW-1466] ability to take joint gains in through a parameter file (#516)
## Change Overview

1. standardizes gain names in the hardware interface to `k_q_p` and `k_qd_p`, same as spot sdk (https://dev.bostondynamics.com/docs/concepts/joint_control/readme)

2. allows taking in `k_q_p` and `k_qd_p` through a a parameter file. If you have a yaml that looks like this
```
/**:
  ros__parameters:
    k_q_p: [624.0, 936.0, 286.0,  624.0, 936.0, 286.0, 624.0, 936.0, 286.0, 624.0, 936.0, 286.0, 1020.0, 255.0, 204.0, 102.0, 102.0, 102.0, 16.0]
    k_qd_p: [5.20, 5.20, 2.04, 5.20, 5.20, 2.04, 5.20, 5.20, 2.04, 5.20, 5.20, 2.04, 10.2, 15.3, 10.2, 2.04, 2.04, 2.04, 0.32]
```
and pass it to the `spot_ros2_control.launch.py` launchfile with the arg `config_file:=<file path>`, these gains will get used in the hardware interface to stream commands.
[Because ros2 control hardware interfaces don't have "true" support for parameters, ](https://github.com/ros-controls/ros2_control/issues/347)the gains have to be passed in as a [string through the xacro](https://github.com/ros-controls/ros2_control/blob/cb91599f8f66aaf39b7485a2f7e131157f633474/hardware_interface/include/hardware_interface/hardware_info.hpp#L182), so this also adds a helper function to assist with this conversion back to a usable vector. 

edge case handling:
1. if either of these params isn't set (or no config file is specified) then the default gains are used. 
2. if either the gain lists defined in the parameter file is the wrong number of elements, the hardware interface will fall back to using the default gains, and a warning will be logged about this.

## Testing Done

* The wiggle arm example has some slightly jerky gripper motion using the default gains.
I changed the `k_qd_p` gain for the gripper joint in my parameter file from `0.32` to `1.32` and reran the example, and the gripper looked a lot smoother. 

* Checked edge case handling manually 

### Next steps

The function to translate the gains as a string into a usable vector in the hardware interface should get unit tested (SW-1148)

File: spot_description/urdf/spot.ros2_control.xacro (robot description, xacro)
@@ -19,8 +19,4 @@
                 <param name="max">${effort_max}</param>
             </command_interface>
-            <!-- TODO at some point, this should be a part of the command interface so we can have a
-            one-to-one mapping to the spot sdk implementation. -->
-            <!-- <command_interface name="k_q_p" />
-            <command_interface name="k_qd_p" /> -->
         </joint>
     </xacro:macro>
@@ -52,5 +48,5 @@
             position_min="-1.570" position_max="0.000" velocity_max="100" effort_max="15.3" />
     </xacro:macro>
-    <xacro:macro name="spot_ros2_control" params="interface_type has_arm hostname username password tf_prefix">
+    <xacro:macro name="spot_ros2_control" params="interface_type has_arm hostname username password tf_prefix k_q_p k_qd_p">
         <!-- Currently implements a simple system interface that covers all joints of the robot.
         In the future, we could make different hardware interfaces for the body, arm, etc. -->
@@ -67,4 +63,6 @@
                 <param name="username">$(optenv BOSDYN_CLIENT_USERNAME ${username})</param>
                 <param name="password">$(optenv BOSDYN_CLIENT_PASSWORD ${password})</param>
+                <param name="k_q_p">${k_q_p}</param>
+                <param name="k_qd_p">${k_qd_p}</param>
             </xacro:if>
             </hardware>

File: spot_description/urdf/spot.urdf.xacro (robot description, xacro)
@@ -12,8 +12,9 @@
   <xacro:arg name="add_ros2_control_tag" default="false" />
   <xacro:arg name="hardware_interface_type" default="mock" />
-  <xacro:arg name="tf_prefix" default="" />
   <xacro:arg name="hostname" default="10.0.0.3" />
   <xacro:arg name="username" default="username" />
   <xacro:arg name="password" default="password" />
+  <xacro:arg name="k_q_p" default="" />
+  <xacro:arg name="k_qd_p" default="" />
   <!-- Load Spot -->
   <xacro:load_spot
@@ -28,5 +29,7 @@
                                username="$(arg username)"
                                password="$(arg password)"
-                               tf_prefix="$(arg tf_prefix)" />
+                               tf_prefix="$(arg tf_prefix)"
+                               k_q_p="$(arg k_q_p)"
+                               k_qd_p="$(arg k_qd_p)" />
   </xacro:if>
 </robot>
