Commit message: part of robot model now shows up in rviz. legs are gone

File: spot_ros2_control/xacro/spot_body.xacro (robot description, xacro)
@@ -1,4 +1,5 @@
 <?xml version="1.0"?>
-<robot name="h1" xmlns:xacro="http://www.ros.org/wiki/xacro">
+<robot name="spot" xmlns:xacro="http://www.ros.org/wiki/xacro">
+    <xacro:arg name="has_arm" default="false" />
     <!-- Add ros2control tag-->
     <xacro:arg name="add_ros2control_tag" default="true" />
@@ -7,12 +8,13 @@
     <!-- we create propery object from the arguments to improve usability later on. Arg have less
     options to be used in if statements-->
+    <xacro:property name="has_arm_property" value="$(arg has_arm)" />
     <xacro:property name="add_ros2control_tag_property" value="$(arg add_ros2control_tag)" />
     <xacro:property name="hardware_interface_type_property" value="$(arg hardware_interface_type)" />
-    <!-- The actual macro containing the urdf of the h1-->
-    <xacro:include filename="$(find spot_description)/urdf/spot.urdf.xacro" />
+    <!-- The actual macro containing the urdf of the spot-->
+    <xacro:include filename="$(find spot_description)/urdf/spot_macro.xacro" />
     <xacro:include filename="$(find spot_ros2_control)/xacro/spot_interfaces.ros2_control.xacro" />
     <xacro:include filename="$(find spot_ros2_control)/xacro/spot.ros2_control.xacro" />
     <!-- Adding Spot-->
-    <xacro:load_spot arm="false" tf_prefix=""/>
+    <xacro:load_spot arm="${has_arm_property}" tf_prefix=""/>
     <!-- Adding the ros2control tags without hands-->
     <xacro:if value="${add_ros2control_tag_property}">
