Commit message: two of the legs show up. unclear why

File: spot_ros2_control/xacro/spot.ros2_control.xacro (robot description, xacro)
@@ -1,28 +1,21 @@
 <?xml version="1.0"?>
 <robot xmlns:xacro="http://www.ros.org/wiki/xacro">
-    <!-- <xacro:macro name="spot_ros2_control">
-        <xacro:if value="${hardware_interface_type_property == 'mock'}">
-            <ros2_control name="SpotSystem" type="system">
-                <hardware>
-                    <plugin>spot_ros2_control/SpotMockJointHardwareInterface</plugin>
-                </hardware>
-                <xacro:leg front_or_back="front" left_or_right="left" />
-                <xacro:leg front_or_back="front" left_or_right="right" />
-                <xacro:leg front_or_back="back" left_or_right="left" />
-                <xacro:leg front_or_back="back" left_or_right="right" />
-            </ros2_control>
-        </xacro:if>
-    </xacro:macro> -->
-    <xacro:macro name="spot_interface_ros2_control">
-        <ros2_control name="RobotInterfaceSystem" type="system">
+    <xacro:macro name="spot_ros2_control" params="interface_type">
+        <ros2_control name="SpotSystem" type="system">
             <hardware>
+            <!-- <xacro:if value="${interface_type == 'spot-sdk'}">
+                <plugin>spot_ros2_control/SpotMockJointHardwareInterface</plugin>
+            </xacro:if> -->
+            <xacro:if value="${interface_type == 'mock'}">
                 <plugin>mock_components/GenericSystem</plugin>
                 <param name="mock_sensor_commands">false</param>
                 <param name="state_following_offset">0.0</param>
+            </xacro:if>
             </hardware>
-            <!-- <xacro:leg front_or_back="front" left_or_right="left" />
+            <!-- Add the joints -->
+            <xacro:leg front_or_back="front" left_or_right="left" />
             <xacro:leg front_or_back="front" left_or_right="right" />
             <xacro:leg front_or_back="back" left_or_right="left" />
-            <xacro:leg front_or_back="back" left_or_right="right" /> -->
+            <xacro:leg front_or_back="back" left_or_right="right" />
         </ros2_control>
     </xacro:macro>

File: spot_ros2_control/xacro/spot.urdf.xacro (robot description, xacro)
@@ -19,6 +19,5 @@
     <!-- Adding the ros2control tags without hands-->
     <xacro:if value="${add_ros2control_tag_property}">
-        <!-- <xacro:spot_ros2_control /> -->
-        <xacro:spot_interface_ros2_control />
+        <xacro:spot_ros2_control interface_type="mock"/>
     </xacro:if>
 </robot>

Commit message: typo -- back legs are actually called rear

File: spot_ros2_control/xacro/spot.ros2_control.xacro (robot description, xacro)
@@ -14,8 +14,8 @@
             </hardware>
             <!-- Add the joints -->
-            <xacro:leg front_or_back="front" left_or_right="left" />
-            <xacro:leg front_or_back="front" left_or_right="right" />
-            <xacro:leg front_or_back="back" left_or_right="left" />
-            <xacro:leg front_or_back="back" left_or_right="right" />
+            <xacro:leg front_or_rear="front" left_or_right="left" />
+            <xacro:leg front_or_rear="front" left_or_right="right" />
+            <xacro:leg front_or_rear="rear" left_or_right="left" />
+            <xacro:leg front_or_rear="rear" left_or_right="right" />
         </ros2_control>
     </xacro:macro>

File: spot_ros2_control/xacro/spot_interfaces.ros2_control.xacro (robot description, xacro)
@@ -28,10 +28,10 @@
         </joint>
     </xacro:macro>
-    <xacro:macro name="leg" params="left_or_right front_or_back">
-        <xacro:ros2control_joint joint_name="${front_or_back}_${left_or_right}_hip_x"
+    <xacro:macro name="leg" params="left_or_right front_or_rear">
+        <xacro:ros2control_joint joint_name="${front_or_rear}_${left_or_right}_hip_x"
             position_min="-0.785" position_max="0.785" velocity_max="100" effort_max="100" />
-        <xacro:ros2control_joint joint_name="${front_or_back}_${left_or_right}_hip_y"
+        <xacro:ros2control_joint joint_name="${front_or_rear}_${left_or_right}_hip_y"
             position_min="-0.899" position_max="2.295" velocity_max="100" effort_max="100" />
-        <xacro:ros2control_joint joint_name="${front_or_back}_${left_or_right}_knee"
+        <xacro:ros2control_joint joint_name="${front_or_rear}_${left_or_right}_knee"
             position_min="-2.793" position_max="-0.255" velocity_max="100" effort_max="100" />
     </xacro:macro>

Commit message: make the interfaces match more with the spot sdk format

File: spot_ros2_control/xacro/spot.ros2_control.xacro (robot description, xacro)
@@ -4,6 +4,7 @@
         <ros2_control name="SpotSystem" type="system">
             <hardware>
+            <!-- TODO: This custom plugin (does not exist yet) can be the one interacting with the spot sdk. -->
             <!-- <xacro:if value="${interface_type == 'spot-sdk'}">
-                <plugin>spot_ros2_control/SpotMockJointHardwareInterface</plugin>
+                <plugin>spot_ros2_control/SpotJointHardwareInterface</plugin>
             </xacro:if> -->
             <xacro:if value="${interface_type == 'mock'}">

File: spot_ros2_control/xacro/spot.urdf.xacro (robot description, xacro)
@@ -2,22 +2,20 @@
 <robot name="spot" xmlns:xacro="http://www.ros.org/wiki/xacro">
     <xacro:arg name="has_arm" default="false" />
-    <!-- Add ros2control tag-->
-    <xacro:arg name="add_ros2control_tag" default="true" />
-    <!-- Add ros2control tag-->
+    <xacro:arg name="add_ros2_control_tag" default="true" />
     <xacro:arg name="hardware_interface_type" default="mock" />
-    <!-- we create propery object from the arguments to improve usability later on. Arg have less
-    options to be used in if statements-->
+    <!-- Create property object from the arguments to improve usability later on -->
     <xacro:property name="has_arm_property" value="$(arg has_arm)" />
-    <xacro:property name="add_ros2control_tag_property" value="$(arg add_ros2control_tag)" />
+    <xacro:property name="add_ros2_control_tag_property" value="$(arg add_ros2_control_tag)" />
     <xacro:property name="hardware_interface_type_property" value="$(arg hardware_interface_type)" />
-    <!-- The actual macro containing the urdf of the spot-->
+    <!-- Macro containing the URDF for Spot -->
     <xacro:include filename="$(find spot_description)/urdf/spot_macro.xacro" />
+    <!-- Macros for loading the ROS 2 control tags -->
     <xacro:include filename="$(find spot_ros2_control)/xacro/spot_interfaces.ros2_control.xacro" />
     <xacro:include filename="$(find spot_ros2_control)/xacro/spot.ros2_control.xacro" />
     <!-- Adding Spot-->
     <xacro:load_spot arm="${has_arm_property}" tf_prefix=""/>
-    <!-- Adding the ros2control tags without hands-->
-    <xacro:if value="${add_ros2control_tag_property}">
-        <xacro:spot_ros2_control interface_type="mock"/>
+    <!-- Adding the ROS 2 control tags -->
+    <xacro:if value="${add_ros2_control_tag_property}">
+        <xacro:spot_ros2_control interface_type="${hardware_interface_type_property}"/>
     </xacro:if>
 </robot>

File: spot_ros2_control/xacro/spot_interfaces.ros2_control.xacro (robot description, xacro)
@@ -1,15 +1,15 @@
 <?xml version="1.0"?>
 <robot xmlns:xacro="http://www.ros.org/wiki/xacro">
-    <xacro:macro name="ros2control_joint"
-        params="joint_name position_min:=0.0 position_max:=0.0 velocity_max effort_max">
+    <xacro:macro name="ros2_control_joint"
+        params="joint_name position_min:=0.0 position_max:=0.0 velocity_max load_max">
         <joint name="${joint_name}">
             <state_interface name="position" />
             <state_interface name="velocity" />
-            <state_interface name="effort" />
+            <state_interface name="load" />
             <state_interface name="position_commanded" />
             <state_interface name="velocity_commanded" />
-            <state_interface name="effort_commanded" />
-            <state_interface name="p_gain_commanded" />
-            <state_interface name="d_gain_commanded" />
+            <state_interface name="load_commanded" />
+            <state_interface name="k_q_p_commanded" />
+            <state_interface name="k_qd_p_commanded" />
             <command_interface name="position">
                 <param name="min">${position_min}</param>
@@ -20,19 +20,20 @@
                 <param name="max">${velocity_max}</param>
             </command_interface>
-            <command_interface name="effort">
-                <param name="min">${-effort_max}</param>
-                <param name="max">${effort_max}</param>
+            <command_interface name="load">
+                <param name="min">${-load_max}</param>
+                <param name="max">${load_max}</param>
             </command_interface>
-            <command_interface name="p_gain" />
-            <command_interface name="d_gain" />
+            <command_interface name="k_q_p" />
+            <command_interface name="k_qd_p" />
         </joint>
     </xacro:macro>
+    <!-- TODO: find actual velocity and load bounds. -->
     <xacro:macro name="leg" params="left_or_right front_or_rear">
-        <xacro:ros2control_joint joint_name="${front_or_rear}_${left_or_right}_hip_x"
-            position_min="-0.785" position_max="0.785" velocity_max="100" effort_max="100" />
-        <xacro:ros2control_joint joint_name="${front_or_rear}_${left_or_right}_hip_y"
-            position_min="-0.899" position_max="2.295" velocity_max="100" effort_max="100" />
-        <xacro:ros2control_joint joint_name="${front_or_rear}_${left_or_right}_knee"
-            position_min="-2.793" position_max="-0.255" velocity_max="100" effort_max="100" />
+        <xacro:ros2_control_joint joint_name="${front_or_rear}_${left_or_right}_hip_x"
+            position_min="-0.785" position_max="0.785" velocity_max="100" load_max="100" />
+        <xacro:ros2_control_joint joint_name="${front_or_rear}_${left_or_right}_hip_y"
+            position_min="-0.899" position_max="2.295" velocity_max="100" load_max="100" />
+        <xacro:ros2_control_joint joint_name="${front_or_rear}_${left_or_right}_knee"
+            position_min="-2.793" position_max="-0.255" velocity_max="100" load_max="100" />
     </xacro:macro>
 </robot>

Commit message: Test launchfiles for squat and arm wiggle

File: spot_ros2_control/xacro/spot.ros2_control.xacro (robot description, xacro)
@@ -1,5 +1,5 @@
 <?xml version="1.0"?>
 <robot xmlns:xacro="http://www.ros.org/wiki/xacro">
-    <xacro:macro name="spot_ros2_control" params="interface_type">
+    <xacro:macro name="spot_ros2_control" params="interface_type has_arm">
         <ros2_control name="SpotSystem" type="system">
             <hardware>
@@ -14,9 +14,13 @@
             </xacro:if>
             </hardware>
-            <!-- Add the joints -->
+            <!-- Add the legs -->
             <xacro:leg front_or_rear="front" left_or_right="left" />
             <xacro:leg front_or_rear="front" left_or_right="right" />
             <xacro:leg front_or_rear="rear" left_or_right="left" />
             <xacro:leg front_or_rear="rear" left_or_right="right" />
+            <!-- Add the arm + the gripper if the robot has an arm -->
+            <xacro:if value="${has_arm}">
+                <xacro:arm/>
+            </xacro:if>
         </ros2_control>
     </xacro:macro>

File: spot_ros2_control/xacro/spot.urdf.xacro (robot description, xacro)
@@ -17,5 +17,5 @@
     <!-- Adding the ROS 2 control tags -->
     <xacro:if value="${add_ros2_control_tag_property}">
-        <xacro:spot_ros2_control interface_type="${hardware_interface_type_property}"/>
+        <xacro:spot_ros2_control interface_type="${hardware_interface_type_property}" has_arm="${has_arm_property}"/>
     </xacro:if>
 </robot>

File: spot_ros2_control/xacro/spot_interfaces.ros2_control.xacro (robot description, xacro)
@@ -37,3 +37,21 @@
             position_min="-2.793" position_max="-0.255" velocity_max="100" load_max="100" />
     </xacro:macro>
+    <xacro:macro name="arm">
+        <xacro:ros2_control_joint joint_name="arm_sh0"
+            position_min="-2.168" position_max="3.142" velocity_max="100" load_max="100" />
+        <xacro:ros2_control_joint joint_name="arm_sh1"
+            position_min="-3.142" position_max="0.524" velocity_max="100" load_max="100" />
+        <xacro:ros2_control_joint joint_name="arm_el0"
+            position_min="0.000" position_max="3.142" velocity_max="100" load_max="100" />
+        <xacro:ros2_control_joint joint_name="arm_el1"
+            position_min="-2.793" position_max="2.793" velocity_max="100" load_max="100" />
+        <xacro:ros2_control_joint joint_name="arm_wr0"
+            position_min="-1.833" position_max="1.833" velocity_max="100" load_max="100" />
+        <xacro:ros2_control_joint joint_name="arm_wr1"
+            position_min="-2.880" position_max="2.880" velocity_max="100" load_max="100" />
+        <!-- TODO: this is the gripper joint. This could be its own interface to support robotsd
+        with custom grippers, but would involve modifying the URDFs in spot description. -->
+        <xacro:ros2_control_joint joint_name="arm_f1x"
+            position_min="-1.570" position_max="0.000" velocity_max="100" load_max="100" />
+    </xacro:macro>
 </robot>

Commit message: Passing in login info one by one

File: spot_ros2_control/xacro/spot.ros2_control.xacro (robot description, xacro)
@@ -1,5 +1,5 @@
 <?xml version="1.0"?>
 <robot xmlns:xacro="http://www.ros.org/wiki/xacro">
-    <xacro:macro name="spot_ros2_control" params="interface_type has_arm">
+    <xacro:macro name="spot_ros2_control" params="interface_type has_arm hostname username password config_file">
         <!-- Currently implements a simple system interface that covers all joints of the robot.
         In the future, we could make different hardware interfaces for the body, arm, etc. -->
@@ -16,4 +16,14 @@
                 <param name="example_param_hw_stop_duration_sec">3.0</param>
                 <param name="example_param_hw_slowdown">100</param>
+                <!-- <xacro:property name="yaml_file" value="$(arg config_file)"/>
+                <param name="test" value="${yaml_file}"/>
+                <xacro:property name="yaml_dict" value="${xacro.load_yaml(yaml_file)}"/>
+                <xacro:property name="ros_params" value="${yaml_dict['/**']['ros__parameters']}"/> -->
+                <xacro:property name="hostname_property" value="$(optenv SPOT_IP ${hostname})"/>
+                <xacro:property name="username_property" value="$(optenv BOSDYN_CLIENT_USERNAME ${username})"/>
+                <xacro:property name="password_property" value="$(optenv BOSDYN_CLIENT_PASSWORD ${password})"/>
+                <param name="hostname">${hostname_property}</param>
+                <param name="username">${username_property}</param>
+                <param name="password">${password_property}</param>
             </xacro:if>
             </hardware>

File: spot_ros2_control/xacro/spot.urdf.xacro (robot description, xacro)
@@ -4,8 +4,13 @@
     <xacro:arg name="add_ros2_control_tag" default="true" />
     <xacro:arg name="hardware_interface_type" default="mock" />
+    <xacro:arg name="hostname" default="10.0.0.3" />
+    <xacro:arg name="username" default="username" />
+    <xacro:arg name="password" default="password" />
+    <xacro:arg name="config_file" default="$(find spot_ros2_control)/config/spot_params.yaml" />
     <!-- Create property object from the arguments to improve usability later on -->
     <xacro:property name="has_arm_property" value="$(arg has_arm)" />
     <xacro:property name="add_ros2_control_tag_property" value="$(arg add_ros2_control_tag)" />
     <xacro:property name="hardware_interface_type_property" value="$(arg hardware_interface_type)" />
+    <xacro:property name="config_file_property" value="$(arg config_file)" />
     <!-- Macro containing the URDF for Spot -->
     <xacro:include filename="$(find spot_description)/urdf/spot_macro.xacro" />
@@ -17,5 +22,10 @@
     <!-- Adding the ROS 2 control tags -->
     <xacro:if value="${add_ros2_control_tag_property}">
-        <xacro:spot_ros2_control interface_type="${hardware_interface_type_property}" has_arm="${has_arm_property}"/>
+        <xacro:spot_ros2_control interface_type="${hardware_interface_type_property}"
+                                 has_arm="${has_arm_property}"
+                                 hostname="$(arg hostname)"
+                                 username="$(arg username)"
+                                 password="$(arg password)"
+                                 config_file="${config_file_property}"/>
     </xacro:if>
 </robot>

Commit message: code cleanup

File: spot_ros2_control/xacro/spot.ros2_control.xacro (robot description, xacro)
@@ -1,5 +1,5 @@
 <?xml version="1.0"?>
 <robot xmlns:xacro="http://www.ros.org/wiki/xacro">
-    <xacro:macro name="spot_ros2_control" params="interface_type has_arm hostname username password config_file">
+    <xacro:macro name="spot_ros2_control" params="interface_type has_arm hostname username password">
         <!-- Currently implements a simple system interface that covers all joints of the robot.
         In the future, we could make different hardware interfaces for the body, arm, etc. -->
@@ -13,17 +13,9 @@
             <xacro:if value="${interface_type == 'spot-sdk'}">
                 <plugin>spot_ros2_control/SpotHardware</plugin>
-                <param name="example_param_hw_start_duration_sec">0</param>
-                <param name="example_param_hw_stop_duration_sec">3.0</param>
-                <param name="example_param_hw_slowdown">100</param>
-                <!-- <xacro:property name="yaml_file" value="$(arg config_file)"/>
-                <param name="test" value="${yaml_file}"/>
-                <xacro:property name="yaml_dict" value="${xacro.load_yaml(yaml_file)}"/>
-                <xacro:property name="ros_params" value="${yaml_dict['/**']['ros__parameters']}"/> -->
-                <xacro:property name="hostname_property" value="$(optenv SPOT_IP ${hostname})"/>
-                <xacro:property name="username_property" value="$(optenv BOSDYN_CLIENT_USERNAME ${username})"/>
-                <xacro:property name="password_property" value="$(optenv BOSDYN_CLIENT_PASSWORD ${password})"/>
-                <param name="hostname">${hostname_property}</param>
-                <param name="username">${username_property}</param>
-                <param name="password">${password_property}</param>
+                <!-- eventually it would be ideal to be able to optionally load these from yaml as well (with
+                xacro.load_yaml) as we support putting the login info into a config file in the spot driver.-->
+                <param name="hostname">$(optenv SPOT_IP ${hostname})</param>
+                <param name="username">$(optenv BOSDYN_CLIENT_USERNAME ${username})</param>
+                <param name="password">$(optenv BOSDYN_CLIENT_PASSWORD ${password})</param>
             </xacro:if>
             </hardware>

File: spot_ros2_control/xacro/spot.urdf.xacro (robot description, xacro)
@@ -7,10 +7,4 @@
     <xacro:arg name="username" default="username" />
     <xacro:arg name="password" default="password" />
-    <xacro:arg name="config_file" default="$(find spot_ros2_control)/config/spot_params.yaml" />
-    <!-- Create property object from the arguments to improve usability later on -->
-    <xacro:property name="has_arm_property" value="$(arg has_arm)" />
-    <xacro:property name="add_ros2_control_tag_property" value="$(arg add_ros2_control_tag)" />
-    <xacro:property name="hardware_interface_type_property" value="$(arg hardware_interface_type)" />
-    <xacro:property name="config_file_property" value="$(arg config_file)" />
     <!-- Macro containing the URDF for Spot -->
     <xacro:include filename="$(find spot_description)/urdf/spot_macro.xacro" />
@@ -19,13 +13,12 @@
     <xacro:include filename="$(find spot_ros2_control)/xacro/spot.ros2_control.xacro" />
     <!-- Adding Spot-->
-    <xacro:load_spot arm="${has_arm_property}" tf_prefix=""/>
+    <xacro:load_spot arm="$(arg has_arm)" tf_prefix=""/>
     <!-- Adding the ROS 2 control tags -->
-    <xacro:if value="${add_ros2_control_tag_property}">
-        <xacro:spot_ros2_control interface_type="${hardware_interface_type_property}"
-                                 has_arm="${has_arm_property}"
+    <xacro:if value="$(arg add_ros2_control_tag)">
+        <xacro:spot_ros2_control interface_type="$(arg hardware_interface_type)"
+                                 has_arm="$(arg has_arm)"
                                  hostname="$(arg hostname)"
                                  username="$(arg username)"
-                                 password="$(arg password)"
-                                 config_file="${config_file_property}"/>
+                                 password="$(arg password)" />
     </xacro:if>
 </robot>
