Commit message: [SW-1237] hardware interface for streaming robot state (#431)
## Change Overview

This PR adds a hardware interface that uses the spot-sdk to broadcast the joint states of the robot. The ability to take in commands will be implemented afterwards. 

Since this is going into a dev branch, the structure could be subject to change (and there are some things here that will need more work), but this gives a baseline for us to build on for the upcoming work.

## Testing Done

- [x] Ran `ros2 launch spot_ros2_control spot_ros2_control.launch.py has_arm:=true controllers_config:=spot_controllers_with_arm.yaml hardware_interface:=spot-sdk` while connected to the robot over ethernet, with the login information specified in my environment variables. The joint state publisher is updated with valid information from the spot sdk, and the robot's position is visible in rviz (see below!)

![Screenshot from 2024-07-25 14-31-56.png](https://graphite-user-uploaded-assets-prod.s3.amazonaws.com/Xynj6CBpA3NqqBFfE8Q9/14f644b3-2a8f-4fbd-a714-72887ada4853.png)

## Things to be addressed in future PRs
* adding command streaming!
* CTRL+C does not deactivate + shutdown the hardware interface, meaning the lease does not get cleanly returned (here this is fine since state streaming doesn't require this). we shouldn't have to manually `ros2 control set_hardware_component_state SpotSystem inactive` when we want to stop the program.
* We should be able to put login info in a yaml (as this is supported in spot driver) that then gets passed to the xacro, then into the hardware interface.

File: spot_ros2_control/xacro/spot.ros2_control.xacro (robot description, xacro)
@@ -1,5 +1,5 @@
 <?xml version="1.0"?>
 <robot xmlns:xacro="http://www.ros.org/wiki/xacro">
-    <xacro:macro name="spot_ros2_control" params="interface_type has_arm">
+    <xacro:macro name="spot_ros2_control" params="interface_type has_arm hostname username password">
         <!-- Currently implements a simple system interface that covers all joints of the robot.
         In the future, we could make different hardware interfaces for the body, arm, etc. -->
@@ -11,9 +11,12 @@
                 <param name="state_following_offset">0.0</param>
             </xacro:if>
-            <!-- TODO Make a custom plugin that interacts with the spot sdk. -->
-            <!-- <xacro:if value="${interface_type == 'spot-sdk'}">
-                <plugin>spot_ros2_control/SpotJointHardwareInterface</plugin>
-                    <param> ....
-            </xacro:if> -->
+            <xacro:if value="${interface_type == 'spot-sdk'}">
+                <plugin>spot_ros2_control/SpotHardware</plugin>
+                <!-- eventually it would be ideal to be able to optionally load these from yaml as well (with
+                xacro.load_yaml) as we support putting the login info into a config file in the spot driver.-->
+                <param name="hostname">$(optenv SPOT_IP ${hostname})</param>
+                <param name="username">$(optenv BOSDYN_CLIENT_USERNAME ${username})</param>
+                <param name="password">$(optenv BOSDYN_CLIENT_PASSWORD ${password})</param>
+            </xacro:if>
             </hardware>
             <!-- Add the legs -->

File: spot_ros2_control/xacro/spot.urdf.xacro (robot description, xacro)
@@ -4,8 +4,7 @@
     <xacro:arg name="add_ros2_control_tag" default="true" />
     <xacro:arg name="hardware_interface_type" default="mock" />
-    <!-- Create property object from the arguments to improve usability later on -->
-    <xacro:property name="has_arm_property" value="$(arg has_arm)" />
-    <xacro:property name="add_ros2_control_tag_property" value="$(arg add_ros2_control_tag)" />
-    <xacro:property name="hardware_interface_type_property" value="$(arg hardware_interface_type)" />
+    <xacro:arg name="hostname" default="10.0.0.3" />
+    <xacro:arg name="username" default="username" />
+    <xacro:arg name="password" default="password" />
     <!-- Macro containing the URDF for Spot -->
     <xacro:include filename="$(find spot_description)/urdf/spot_macro.xacro" />
@@ -14,8 +13,12 @@
     <xacro:include filename="$(find spot_ros2_control)/xacro/spot.ros2_control.xacro" />
     <!-- Adding Spot-->
-    <xacro:load_spot arm="${has_arm_property}" tf_prefix=""/>
+    <xacro:load_spot arm="$(arg has_arm)" tf_prefix=""/>
     <!-- Adding the ROS 2 control tags -->
-    <xacro:if value="${add_ros2_control_tag_property}">
-        <xacro:spot_ros2_control interface_type="${hardware_interface_type_property}" has_arm="${has_arm_property}"/>
+    <xacro:if value="$(arg add_ros2_control_tag)">
+        <xacro:spot_ros2_control interface_type="$(arg hardware_interface_type)"
+                                 has_arm="$(arg has_arm)"
+                                 hostname="$(arg hostname)"
+                                 username="$(arg username)"
+                                 password="$(arg password)" />
     </xacro:if>
 </robot>

File: spot_ros2_control/xacro/spot_interfaces.ros2_control.xacro (robot description, xacro)
@@ -1,5 +1,4 @@
 <?xml version="1.0"?>
 <robot xmlns:xacro="http://www.ros.org/wiki/xacro">
-    <!-- The interfaces in this are modeled after the parameters from low level control in the spot sdk. -->
     <xacro:macro name="ros2_control_joint"
         params="joint_name position_min:=0.0 position_max:=0.0 velocity_max effort_max">
@@ -8,9 +7,4 @@
             <state_interface name="velocity" />
             <state_interface name="effort" />
-            <state_interface name="position_commanded" />
-            <state_interface name="velocity_commanded" />
-            <state_interface name="effort_commanded" />
-            <state_interface name="k_q_p_commanded" />
-            <state_interface name="k_qd_p_commanded" />
             <command_interface name="position">
                 <param name="min">${position_min}</param>
@@ -25,6 +19,8 @@
                 <param name="max">${effort_max}</param>
             </command_interface>
-            <command_interface name="k_q_p" />
-            <command_interface name="k_qd_p" />
+            <!-- TODO at some point, this should be a part of the command interface so we can have a
+            one-to-one mapping to the spot sdk implementation. -->
+            <!-- <command_interface name="k_q_p" />
+            <command_interface name="k_qd_p" /> -->
         </joint>
     </xacro:macro>

Commit message: Working omg

File: spot_ros2_control/xacro/spot.ros2_control.xacro (robot description, xacro)
@@ -1,5 +1,5 @@
 <?xml version="1.0"?>
 <robot xmlns:xacro="http://www.ros.org/wiki/xacro">
-    <xacro:macro name="spot_ros2_control" params="interface_type has_arm hostname username password">
+    <xacro:macro name="spot_ros2_control" params="interface_type has_arm hostname username password tf_prefix">
         <!-- Currently implements a simple system interface that covers all joints of the robot.
         In the future, we could make different hardware interfaces for the body, arm, etc. -->
@@ -19,11 +19,11 @@
             </hardware>
             <!-- Add the legs -->
-            <xacro:leg front_or_rear="front" left_or_right="left" />
-            <xacro:leg front_or_rear="front" left_or_right="right" />
-            <xacro:leg front_or_rear="rear" left_or_right="left" />
-            <xacro:leg front_or_rear="rear" left_or_right="right" />
+            <xacro:leg front_or_rear="front" left_or_right="left" tf_prefix="${tf_prefix}" />
+            <xacro:leg front_or_rear="front" left_or_right="right" tf_prefix="${tf_prefix}" />
+            <xacro:leg front_or_rear="rear" left_or_right="left" tf_prefix="${tf_prefix}" />
+            <xacro:leg front_or_rear="rear" left_or_right="right" tf_prefix="${tf_prefix}" />
             <!-- Add the arm + the gripper if the robot has an arm -->
             <xacro:if value="${has_arm}">
-                <xacro:arm/>
+                <xacro:arm tf_prefix="${tf_prefix}" />
             </xacro:if>
         </ros2_control>

File: spot_ros2_control/xacro/spot.urdf.xacro (robot description, xacro)
@@ -4,4 +4,5 @@
     <xacro:arg name="add_ros2_control_tag" default="true" />
     <xacro:arg name="hardware_interface_type" default="mock" />
+    <xacro:arg name="tf_prefix" default="" />
     <xacro:arg name="hostname" default="10.0.0.3" />
     <xacro:arg name="username" default="username" />
@@ -13,5 +14,5 @@
     <xacro:include filename="$(find spot_ros2_control)/xacro/spot.ros2_control.xacro" />
     <!-- Adding Spot-->
-    <xacro:load_spot arm="$(arg has_arm)" tf_prefix=""/>
+    <xacro:load_spot arm="$(arg has_arm)" tf_prefix="$(arg tf_prefix)"/>
     <!-- Adding the ROS 2 control tags -->
     <xacro:if value="$(arg add_ros2_control_tag)">
@@ -20,5 +21,6 @@
                                  hostname="$(arg hostname)"
                                  username="$(arg username)"
-                                 password="$(arg password)" />
+                                 password="$(arg password)"
+                                 tf_prefix="$(arg tf_prefix)" />
     </xacro:if>
 </robot>

File: spot_ros2_control/xacro/spot_interfaces.ros2_control.xacro (robot description, xacro)
@@ -26,28 +26,28 @@
     </xacro:macro>
     <!-- TODO We do not know the real velocity bounds for Spot. -->
-    <xacro:macro name="leg" params="left_or_right front_or_rear">
-        <xacro:ros2_control_joint joint_name="${front_or_rear}_${left_or_right}_hip_x"
+    <xacro:macro name="leg" params="left_or_right front_or_rear tf_prefix">
+        <xacro:ros2_control_joint joint_name="${tf_prefix}${front_or_rear}_${left_or_right}_hip_x"
             position_min="-0.785" position_max="0.785" velocity_max="100" effort_max="45" />
-        <xacro:ros2_control_joint joint_name="${front_or_rear}_${left_or_right}_hip_y"
+        <xacro:ros2_control_joint joint_name="${tf_prefix}${front_or_rear}_${left_or_right}_hip_y"
             position_min="-0.899" position_max="2.295" velocity_max="100" effort_max="45" />
-        <xacro:ros2_control_joint joint_name="${front_or_rear}_${left_or_right}_knee"
+        <xacro:ros2_control_joint joint_name="${tf_prefix}${front_or_rear}_${left_or_right}_knee"
             position_min="-2.793" position_max="-0.255" velocity_max="100" effort_max="115" />
     </xacro:macro>
-    <xacro:macro name="arm">
-        <xacro:ros2_control_joint joint_name="arm_sh0"
+    <xacro:macro name="arm" params="tf_prefix">
+        <xacro:ros2_control_joint joint_name="${tf_prefix}arm_sh0"
             position_min="-2.168" position_max="3.142" velocity_max="100" effort_max="90.9" />
-        <xacro:ros2_control_joint joint_name="arm_sh1"
+        <xacro:ros2_control_joint joint_name="${tf_prefix}arm_sh1"
             position_min="-3.142" position_max="0.524" velocity_max="100" effort_max="181.8" />
-        <xacro:ros2_control_joint joint_name="arm_el0"
+        <xacro:ros2_control_joint joint_name="${tf_prefix}arm_el0"
             position_min="0.000" position_max="3.142" velocity_max="100" effort_max="90.9" />
-        <xacro:ros2_control_joint joint_name="arm_el1"
+        <xacro:ros2_control_joint joint_name="${tf_prefix}arm_el1"
             position_min="-2.793" position_max="2.793" velocity_max="100" effort_max="30.3" />
-        <xacro:ros2_control_joint joint_name="arm_wr0"
+        <xacro:ros2_control_joint joint_name="${tf_prefix}arm_wr0"
             position_min="-1.833" position_max="1.833" velocity_max="100" effort_max="30.3" />
-        <xacro:ros2_control_joint joint_name="arm_wr1"
+        <xacro:ros2_control_joint joint_name="${tf_prefix}arm_wr1"
             position_min="-2.880" position_max="2.880" velocity_max="100" effort_max="30.3" />
         <!-- This is the gripper joint. This could be its own interface to support robots
         with custom grippers, but would involve modifying the URDFs in spot_description. -->
-        <xacro:ros2_control_joint joint_name="arm_f1x"
+        <xacro:ros2_control_joint joint_name="${tf_prefix}arm_f1x"
             position_min="-1.570" position_max="0.000" velocity_max="100" effort_max="15.3" />
     </xacro:macro>
