Commit message: [SW-1175] ros2_control framework with mock hardware interface (#426)
Adds a framework for working on low level control of spot with ros2 control.

Currently, this adds a mock hardware interface to Spot's URDF and a forward position controller. This includes main launchfile `ros2 launch spot_ros2_control spot_ros2_control.launch.py` to bring up the ros2 control nodes for Spot.

Additionally, there are two nodes that use the forward position controller to move Spot's joints based off the Boston Dynamics SDK examples `noarm_squat` and `wiggle_arm` (https://github.com/boston-dynamics/spot-cpp-sdk/tree/master/cpp/examples/joint_control). They can be launched with `ros2 launch spot_ros2_control test_noarm_squat.launch.py` and `ros2 launch spot_ros2_control test_wiggle_arm.launch.py`. These are mainly meant as a proof of concept to show that the entire stack is functional.

- [x] Test launchfiles successfully load the desired hardware interface and controller, and are able to move the joints
- [x] successfully builds and runs both inside and outside our internal docker

File: spot_ros2_control/xacro/spot_interfaces.ros2_control.xacro (robot description, xacro)
@@ -53,2 +53,60 @@
     </xacro:macro>
 </robot>
+<?xml version="1.0"?>
+<robot xmlns:xacro="http://www.ros.org/wiki/xacro">
+    <!-- The interfaces in this are modeled after the parameters from low level control in the spot sdk. -->
+    <xacro:macro name="ros2_control_joint"
+        params="joint_name position_min:=0.0 position_max:=0.0 velocity_max effort_max">
+        <joint name="${joint_name}">
+            <state_interface name="position" />
+            <state_interface name="velocity" />
+            <state_interface name="effort" />
+            <state_interface name="position_commanded" />
+            <state_interface name="velocity_commanded" />
+            <state_interface name="effort_commanded" />
+            <state_interface name="k_q_p_commanded" />
+            <state_interface name="k_qd_p_commanded" />
+            <command_interface name="position">
+                <param name="min">${position_min}</param>
+                <param name="max">${position_max}</param>
+            </command_interface>
+            <command_interface name="velocity">
+                <param name="min">${-velocity_max}</param>
+                <param name="max">${velocity_max}</param>
+            </command_interface>
+            <command_interface name="effort">
+                <param name="min">${-effort_max}</param>
+                <param name="max">${effort_max}</param>
+            </command_interface>
+            <command_interface name="k_q_p" />
+            <command_interface name="k_qd_p" />
+        </joint>
+    </xacro:macro>
+    <!-- TODO We do not know the real velocity bounds for Spot. -->
+    <xacro:macro name="leg" params="left_or_right front_or_rear">
+        <xacro:ros2_control_joint joint_name="${front_or_rear}_${left_or_right}_hip_x"
+            position_min="-0.785" position_max="0.785" velocity_max="100" effort_max="45" />
+        <xacro:ros2_control_joint joint_name="${front_or_rear}_${left_or_right}_hip_y"
+            position_min="-0.899" position_max="2.295" velocity_max="100" effort_max="45" />
+        <xacro:ros2_control_joint joint_name="${front_or_rear}_${left_or_right}_knee"
+            position_min="-2.793" position_max="-0.255" velocity_max="100" effort_max="115" />
+    </xacro:macro>
+    <xacro:macro name="arm">
+        <xacro:ros2_control_joint joint_name="arm_sh0"
+            position_min="-2.168" position_max="3.142" velocity_max="100" effort_max="90.9" />
+        <xacro:ros2_control_joint joint_name="arm_sh1"
+            position_min="-3.142" position_max="0.524" velocity_max="100" effort_max="181.8" />
+        <xacro:ros2_control_joint joint_name="arm_el0"
+            position_min="0.000" position_max="3.142" velocity_max="100" effort_max="90.9" />
+        <xacro:ros2_control_joint joint_name="arm_el1"
+            position_min="-2.793" position_max="2.793" velocity_max="100" effort_max="30.3" />
+        <xacro:ros2_control_joint joint_name="arm_wr0"
+            position_min="-1.833" position_max="1.833" velocity_max="100" effort_max="30.3" />
+        <xacro:ros2_control_joint joint_name="arm_wr1"
+            position_min="-2.880" position_max="2.880" velocity_max="100" effort_max="30.3" />
+        <!-- This is the gripper joint. This could be its own interface to support robots
+        with custom grippers, but would involve modifying the URDFs in spot_description. -->
+        <xacro:ros2_control_joint joint_name="arm_f1x"
+            position_min="-1.570" position_max="0.000" velocity_max="100" effort_max="15.3" />
+    </xacro:macro>
+</robot>

Commit message: [SW-1322] Namespacing support for spot_ros2_control (#461)
This PR adds namespacing for the ros2 control nodes that get launched in order to mimic the setup we have in the spot_driver. There is a new launch argument `spot_name` in `spot_ros2_control.launch.py` that will apply a namespace to all of the nodes launched by this stack.

Discovered some fun issues with how ros2 control handles namespacing with respect to the config files for the controllers that get used. The names of the nodes in the config file must match the namespace applied. So a config file that looks like:
```
controller_manager:
  ros__parameters:
    update_rate: 333  # Hz

    joint_state_broadcaster:
      type: joint_state_broadcaster/JointStateBroadcaster
...
```
Does not actually work if you have launched the controller manager in a namespace, say `/spot/controller_manager`. Your config file needs to look like
```
spot/controller_manager:
  ros__parameters:
    update_rate: 333  # Hz

    joint_state_broadcaster:
      type: joint_state_broadcaster/JointStateBroadcaster
...
```
instead.

Putting all of these parameters in the global namespace is also not a good idea, as the config file is designed to hold many different types of controllers. (eg, you would also want to change `forward_position_controller` to `spot/forward_position_controller`, later on in this config, and this could cause issues if there were any parameters that had the same name between these two controllers). So the only solution is to generate a config file with the name appended to it at runtime, and use that. We already have done this in the spot_driver rviz launchfile [here](https://github.com/bdaiinstitute/spot_ros2/blob/main/spot_driver/launch/rviz.launch.py) so this follows that same convention about how to modify a template file and save it. Alongside this, we also have to do the same thing if we want rviz to show the robot in different namespaces too.

- [x] tested in mock mode: `ros2 launch spot_ros2_control spot_ros2_control.launch.py hardware_interface:=mock  mock_has_arm:=false spot_name:=test`
- [x] tested on robot: `ros2 launch spot_ros2_control spot_ros2_control.launch.py config_file:=spot_ros.yaml hardware_interface:=robot spot_name:=test`

Please create a checklist of tests you plan to do and check off the ones that have been completed successfully. Ensure that ROS 2 tests use `domain_coordinator` to prevent port conflicts. Further guidance for testing can be found on the [ros utilities wiki](https://github.com/bdaiinstitute/ros_utilities/wiki/Testing-guidelines).

File: spot_ros2_control/xacro/spot_interfaces.ros2_control.xacro (robot description, xacro)
@@ -84,25 +84,25 @@
         <xacro:ros2_control_joint joint_name="${front_or_rear}_${left_or_right}_hip_x"
             position_min="-0.785" position_max="0.785" velocity_max="100" effort_max="45" />
-        <xacro:ros2_control_joint joint_name="${front_or_rear}_${left_or_right}_hip_y"
+        <xacro:ros2_control_joint joint_name="${tf_prefix}${front_or_rear}_${left_or_right}_hip_y"
             position_min="-0.899" position_max="2.295" velocity_max="100" effort_max="45" />
-        <xacro:ros2_control_joint joint_name="${front_or_rear}_${left_or_right}_knee"
+        <xacro:ros2_control_joint joint_name="${tf_prefix}${front_or_rear}_${left_or_right}_knee"
             position_min="-2.793" position_max="-0.255" velocity_max="100" effort_max="115" />
     </xacro:macro>
-    <xacro:macro name="arm">
-        <xacro:ros2_control_joint joint_name="arm_sh0"
+    <xacro:macro name="arm" params="tf_prefix">
+        <xacro:ros2_control_joint joint_name="${tf_prefix}arm_sh0"
             position_min="-2.168" position_max="3.142" velocity_max="100" effort_max="90.9" />
-        <xacro:ros2_control_joint joint_name="arm_sh1"
+        <xacro:ros2_control_joint joint_name="${tf_prefix}arm_sh1"
             position_min="-3.142" position_max="0.524" velocity_max="100" effort_max="181.8" />
-        <xacro:ros2_control_joint joint_name="arm_el0"
+        <xacro:ros2_control_joint joint_name="${tf_prefix}arm_el0"
             position_min="0.000" position_max="3.142" velocity_max="100" effort_max="90.9" />
-        <xacro:ros2_control_joint joint_name="arm_el1"
+        <xacro:ros2_control_joint joint_name="${tf_prefix}arm_el1"
             position_min="-2.793" position_max="2.793" velocity_max="100" effort_max="30.3" />
-        <xacro:ros2_control_joint joint_name="arm_wr0"
+        <xacro:ros2_control_joint joint_name="${tf_prefix}arm_wr0"
             position_min="-1.833" position_max="1.833" velocity_max="100" effort_max="30.3" />
-        <xacro:ros2_control_joint joint_name="arm_wr1"
+        <xacro:ros2_control_joint joint_name="${tf_prefix}arm_wr1"
             position_min="-2.880" position_max="2.880" velocity_max="100" effort_max="30.3" />
         <!-- This is the gripper joint. This could be its own interface to support robots
         with custom grippers, but would involve modifying the URDFs in spot_description. -->
-        <xacro:ros2_control_joint joint_name="arm_f1x"
+        <xacro:ros2_control_joint joint_name="${tf_prefix}arm_f1x"
             position_min="-1.570" position_max="0.000" velocity_max="100" effort_max="15.3" />
     </xacro:macro>

Commit message: rebase fix

File: spot_ros2_control/xacro/spot_interfaces.ros2_control.xacro (robot description, xacro)
@@ -53,57 +53,2 @@
     </xacro:macro>
 </robot>
-<?xml version="1.0"?>
-<robot xmlns:xacro="http://www.ros.org/wiki/xacro">
-    <!-- The interfaces in this are modeled after the parameters from low level control in the spot sdk. -->
-    <xacro:macro name="ros2_control_joint"
-        params="joint_name position_min:=0.0 position_max:=0.0 velocity_max effort_max">
-        <joint name="${joint_name}">
-            <state_interface name="position" />
-            <state_interface name="velocity" />
-            <state_interface name="effort" />
-            <command_interface name="position">
-                <param name="min">${position_min}</param>
-                <param name="max">${position_max}</param>
-            </command_interface>
-            <command_interface name="velocity">
-                <param name="min">${-velocity_max}</param>
-                <param name="max">${velocity_max}</param>
-            </command_interface>
-            <command_interface name="effort">
-                <param name="min">${-effort_max}</param>
-                <param name="max">${effort_max}</param>
-            </command_interface>
-            <!-- TODO at some point, this should be a part of the command interface so we can have a
-            one-to-one mapping to the spot sdk implementation. -->
-            <!-- <command_interface name="k_q_p" />
-            <command_interface name="k_qd_p" /> -->
-        </joint>
-    </xacro:macro>
-    <!-- TODO We do not know the real velocity bounds for Spot. -->
-    <xacro:macro name="leg" params="left_or_right front_or_rear">
-        <xacro:ros2_control_joint joint_name="${front_or_rear}_${left_or_right}_hip_x"
-            position_min="-0.785" position_max="0.785" velocity_max="100" effort_max="45" />
-        <xacro:ros2_control_joint joint_name="${tf_prefix}${front_or_rear}_${left_or_right}_hip_y"
-            position_min="-0.899" position_max="2.295" velocity_max="100" effort_max="45" />
-        <xacro:ros2_control_joint joint_name="${tf_prefix}${front_or_rear}_${left_or_right}_knee"
-            position_min="-2.793" position_max="-0.255" velocity_max="100" effort_max="115" />
-    </xacro:macro>
-    <xacro:macro name="arm" params="tf_prefix">
-        <xacro:ros2_control_joint joint_name="${tf_prefix}arm_sh0"
-            position_min="-2.168" position_max="3.142" velocity_max="100" effort_max="90.9" />
-        <xacro:ros2_control_joint joint_name="${tf_prefix}arm_sh1"
-            position_min="-3.142" position_max="0.524" velocity_max="100" effort_max="181.8" />
-        <xacro:ros2_control_joint joint_name="${tf_prefix}arm_el0"
-            position_min="0.000" position_max="3.142" velocity_max="100" effort_max="90.9" />
-        <xacro:ros2_control_joint joint_name="${tf_prefix}arm_el1"
-            position_min="-2.793" position_max="2.793" velocity_max="100" effort_max="30.3" />
-        <xacro:ros2_control_joint joint_name="${tf_prefix}arm_wr0"
-            position_min="-1.833" position_max="1.833" velocity_max="100" effort_max="30.3" />
-        <xacro:ros2_control_joint joint_name="${tf_prefix}arm_wr1"
-            position_min="-2.880" position_max="2.880" velocity_max="100" effort_max="30.3" />
-        <!-- This is the gripper joint. This could be its own interface to support robots
-        with custom grippers, but would involve modifying the URDFs in spot_description. -->
-        <xacro:ros2_control_joint joint_name="${tf_prefix}arm_f1x"
-            position_min="-1.570" position_max="0.000" velocity_max="100" effort_max="15.3" />
-    </xacro:macro>
-</robot>
